File: Connector_Extension_Board_V1.0/Connector_Extension_Board_V1.0.kicad_pcb (KiCad board)
At the start: 4 copper layers, 67.7 x 69 mm, 11 parts

Commit message: Hoan thanh footprint
Parts:
- removed 12V, 5V, GND: TestPoint_THTPad_3.0x3.0mm_Drill1.5mm, TestPoint:TestPoint_THTPad_3.0x3.0mm_Drill1.5mm
- removed Compute1: Conn_01x02, Library:TE_5-104809-1
- removed Winch2, Winch3, Winch4, Winch5: Conn_01x02, Library:MOLEX_1722871102
- added C10: 120n/50V/0603, Capacitor_SMD:C_0603_1608Metric, F.Cu at (127.4, 90.4)
- added C11: 120n/50V/0603, Capacitor_SMD:C_0603_1608Metric, F.Cu at (155.7, 74.1)
- added C12: 10u/50V/1206, Capacitor_SMD:C_1206_3216Metric, F.Cu at (108.4, 88.2)
- added C13: 120n/50V/0603, Capacitor_SMD:C_0603_1608Metric, F.Cu at (105.4, 90.3)
- added C14: 10u/50V/1206, Capacitor_SMD:C_1206_3216Metric, F.Cu at (119.7, 88.2)
- added C15: 10u/50V/1206, Capacitor_SMD:C_1206_3216Metric, F.Cu at (149.2, 69.9)
- added C16: 10u/50V/1206, Capacitor_SMD:C_1206_3216Metric, F.Cu at (141.7, 96.9)
- added C17: 10u/50V/1206, Capacitor_SMD:C_1206_3216Metric, F.Cu at (108.4, 70.6)
- added C18: 120n/50V/0603, Capacitor_SMD:C_0603_1608Metric, F.Cu at (116.9, 90.3)
- added C19: 10u/50V/1206, Capacitor_SMD:C_1206_3216Metric, F.Cu at (108.5, 96.9)
- added C20: 120n/50V/0603, Capacitor_SMD:C_0603_1608Metric, F.Cu at (105.6, 72.5)
- added C21: 10u/50V/1206, Capacitor_SMD:C_1206_3216Metric, F.Cu at (119.7, 96.8)
- added C22: 10u/50V/1206, Capacitor_SMD:C_1206_3216Metric, F.Cu at (108.3, 79.0)
- added C26: 100nF/50V/0603, Capacitor_SMD:C_0603_1608Metric, F.Cu at (155.3, 97.9)
- added C27: 10u/50V/1206, Capacitor_SMD:C_1206_3216Metric, F.Cu at (130.2, 96.7)
- added C28: 10u/50V/1206, Capacitor_SMD:C_1206_3216Metric, F.Cu at (158.5, 80.6)
- added C4: 10u/50V/1206, Capacitor_SMD:C_1206_3216Metric, F.Cu at (140.7, 69.8)
- added C5: 10u/50V/1206, Capacitor_SMD:C_1206_3216Metric, F.Cu at (141.6, 88.3)
- added C6: 10u/50V/1206, Capacitor_SMD:C_1206_3216Metric, F.Cu at (158.6, 72.1)
- added C7: 10u/50V/1206, Capacitor_SMD:C_1206_3216Metric, F.Cu at (130.2, 88.4)
- added C8: 120n/50V/0603, Capacitor_SMD:C_0603_1608Metric, F.Cu at (142.7, 72.7)
- added C9: 120n/50V/0603, Capacitor_SMD:C_0603_1608Metric, F.Cu at (138.9, 90.5)
- added Computer1: 1723103102, Library:MOLEX_1723103102, F.Cu at (156.4, 62.3)
- added J1: 640388-3, Library:TE_640388-3, F.Cu at (123.9, 52.8)
- added Lidar1: 1723103102, Library:MOLEX_1723103102, F.Cu at (140.3, 104.5)
- added R10: 1.8k/0603/1%, Resistor_SMD:R_0603_1608Metric, F.Cu at (105.6, 74.1)
- added R11: 1k/0603/1%, Resistor_SMD:R_0603_1608Metric, F.Cu at (144.3, 66.0)
- added R12: 1k/0603/1%, Resistor_SMD:R_0603_1608Metric, F.Cu at (145.6, 92.0)
- added R13: 1k/0603/1%, Resistor_SMD:R_0603_1608Metric, F.Cu at (134.1, 92.0)
- added R16: 1k/0603/1%, Resistor_SMD:R_0603_1608Metric, F.Cu at (112.3, 92.1)
- added R17: 1k/0603/1%, Resistor_SMD:R_0603_1608Metric, F.Cu at (112.3, 74.1)
- added R19: 1k/0603/1%, Resistor_SMD:R_0603_1608Metric, F.Cu at (123.6, 92.1)
- added R23: 12.7k/0603/1%, Resistor_SMD:R_0603_1608Metric, F.Cu at (149.6, 90.8)
- added R24: 10k/0603/1%, Resistor_SMD:R_0603_1608Metric, F.Cu at (153.0, 87.2)
- added R25: 1k/0603/1%, Resistor_SMD:R_0603_1608Metric, F.Cu at (149.9, 87.2)
- added R26: 4.99k/0603/1%, Resistor_SMD:R_0603_1608Metric, F.Cu at (151.4, 87.2)
- added R27: 4.99k/0603/1%, Resistor_SMD:R_0603_1608Metric, F.Cu at (154.5, 87.2)
- added R28: 4.99k/0603/1%, Resistor_SMD:R_0603_1608Metric, F.Cu at (156.1, 87.2)
- added R29: 100k/0603/1%, Resistor_SMD:R_0603_1608Metric, F.Cu at (141.2, 66.0)
- added R30: 10.7k/0603/1%, Resistor_SMD:R_0603_1608Metric, F.Cu at (142.8, 66.0)
- added R31: 100k/0603/1%, Resistor_SMD:R_0603_1608Metric, F.Cu at (145.7, 88.9)
- added R32: 10.7k/0603/1%, Resistor_SMD:R_0603_1608Metric, F.Cu at (145.7, 90.4)
- added R33: 100k/0603/1%, Resistor_SMD:R_0603_1608Metric, F.Cu at (134.2, 88.9)
- added R34: 10.7k/0603/1%, Resistor_SMD:R_0603_1608Metric, F.Cu at (134.2, 90.4)
- added R35: 100k/0603/1%, Resistor_SMD:R_0603_1608Metric, F.Cu at (162.5, 72.6)
- added R36: 10.7k/0603/1%, Resistor_SMD:R_0603_1608Metric, F.Cu at (162.5, 74.2)
- added R37: 1k/0603/1%, Resistor_SMD:R_0603_1608Metric, F.Cu at (162.5, 75.7)
- added R38: 100k/0603/1%, Resistor_SMD:R_0603_1608Metric, F.Cu at (112.3, 89.0)
- added R39: 4.87k/0603/1%, Resistor_SMD:R_0603_1608Metric, F.Cu at (112.3, 90.6)
- added R4: 1.8k/0603/1%, Resistor_SMD:R_0603_1608Metric, F.Cu at (144.3, 72.7)
- added R40: 100k/0603/1%, Resistor_SMD:R_0603_1608Metric, F.Cu at (123.6, 89.0)
- added R41: 4.87k/0603/1%, Resistor_SMD:R_0603_1608Metric, F.Cu at (123.6, 90.5)
- added R42: 100k/0603/1%, Resistor_SMD:R_0603_1608Metric, F.Cu at (112.3, 71.0)
- added R43: 4.87k/0603/1%, Resistor_SMD:R_0603_1608Metric, F.Cu at (112.3, 72.6)
- added R5: 2.05k/0603/1%, Resistor_SMD:R_0603_1608Metric, F.Cu at (138.9, 92.0)
- added R6: 6.19k/0603/1%, Resistor_SMD:R_0603_1608Metric, F.Cu at (155.7, 75.7)
- added R7: 2.43k/0603/1%, Resistor_SMD:R_0603_1608Metric, F.Cu at (105.4, 91.8)
- added R8: 4.12k/0603/1%, Resistor_SMD:R_0603_1608Metric, F.Cu at (127.3, 92.0)
- added R9: 1.8k/0603/1%, Resistor_SMD:R_0603_1608Metric, F.Cu at (116.9, 91.9)
- added Spare1: 1723103102, Library:MOLEX_1723103102, F.Cu at (128.9, 104.5)
- added TP1: Lora, Library:TestPoint_Loop_D2.50mm_Drill1.0mm, F.Cu at (161.0, 83.8)
- added TP2: Lora, Library:TestPoint_Loop_D2.50mm_Drill1.0mm, F.Cu at (161.0, 87.7)
- added TP3: Spare, Library:TestPoint_Loop_D2.50mm_Drill1.0mm, F.Cu at (102.6, 83.3)
- added TP4: Spare, Library:TestPoint_Loop_D2.50mm_Drill1.0mm, F.Cu at (102.6, 87.2)
- added U10: SIP32433ADN-T1E4, Library:DFN-10-1EP_3x3mm_P0.5mm_EP1.7x2.5mm, F.Cu at (159.1, 77.1)
- added U11: SIP32433ADN-T1E4, Library:DFN-10-1EP_3x3mm_P0.5mm_EP1.7x2.5mm, F.Cu at (120.2, 93.4)
- added U12: SIP32433ADN-T1E4, Library:DFN-10-1EP_3x3mm_P0.5mm_EP1.7x2.5mm, F.Cu at (108.9, 75.5)
- added U3: SIP32433ADN-T1E4, Library:DFN-10-1EP_3x3mm_P0.5mm_EP1.7x2.5mm, F.Cu at (145.7, 69.4)
- added U4: SIP32433ADN-T1E4, Library:DFN-10-1EP_3x3mm_P0.5mm_EP1.7x2.5mm, F.Cu at (142.3, 93.4)
- added U5: SIP32433ADN-T1E4, Library:DFN-10-1EP_3x3mm_P0.5mm_EP1.7x2.5mm, F.Cu at (130.7, 93.4)
- added U8: SIP32433ADN-T1E4, Library:DFN-10-1EP_3x3mm_P0.5mm_EP1.7x2.5mm, F.Cu at (109.0, 93.4)
- added U9: TPS1HC30BQPWPRQ1, Library:IC_TPS1HC30BQPWPRQ1, F.Cu at (153.4, 93.1)
- GPS1, Phone1: footprint Library:TE_5-104809-1 -> Library:TE_5-104361-1
- Winch1: value Conn_01x02 -> 1723103102; footprint Library:MOLEX_1722871102 -> Library:MOLEX_1723103102
- moved Phone1 10.9 mm to (121.3, 105.1)
- moved GPS1 10.2 mm to (112.3, 105.1)
- moved Winch1 9.34 mm to (151.8, 104.5), turned to 0 degrees
Connections:
- GPS1 pad 1: /5V_REG_2/V_OUT -> /+5V-2A
- Phone1 pad 1: /5V_REG_3/V_OUT -> /+5V-3A_1
- Winch1 pad 1: /WINCH_REG/VOUT -> /+12V-7A
Other:
- board text added: "+"
- board text added: "5V 12V GND"
- board text added: "Compute"
- board text added: "GPS"
- board text added: "Lidar"
- board text added: "Phone"
- board text added: "VIN"
- board text added: "Winch"
- board text removed: "Compute1"
- board text removed: "Encoder"
- board text removed: "GPS1"
- board text removed: "LIDAR1"
- board text removed: "Phone1"
- board text removed: "Winch1"

Commit message: Hoan thanh chinh sua theo phan hoi 12/1
Parts:
- removed R12, R13, R16, R17, R19, R37: 1k/0603/1%, Resistor_SMD:R_0603_1608Metric
- removed R29, R31, R33, R35, R38, R40, R42: 100k/0603/1%, Resistor_SMD:R_0603_1608Metric
- removed R30, R32, R34, R36: 10.7k/0603/1%, Resistor_SMD:R_0603_1608Metric
- removed R39, R41, R43: 4.87k/0603/1%, Resistor_SMD:R_0603_1608Metric
- removed R8: 4.12k/0603/1%, Resistor_SMD:R_0603_1608Metric
- added C23: 3.3nF/50V/0603, Capacitor_SMD:C_0603_1608Metric, F.Cu at (143.3, 67.5)
- added C24: 3.3nF/50V/0603, Capacitor_SMD:C_0603_1608Metric, F.Cu at (143.9, 89.3)
- added C25: 3.3nF/50V/0603, Capacitor_SMD:C_0603_1608Metric, F.Cu at (132.2, 89.3)
- added C29: 3.3nF/50V/0603, Capacitor_SMD:C_0603_1608Metric, F.Cu at (160.7, 73.0)
- added C30: 3.3nF/50V/0603, Capacitor_SMD:C_0603_1608Metric, F.Cu at (110.6, 89.3)
- added C31: 3.3nF/50V/0603, Capacitor_SMD:C_0603_1608Metric, F.Cu at (121.9, 89.3)
- added C32: 3.3nF/50V/0603, Capacitor_SMD:C_0603_1608Metric, F.Cu at (110.4, 71.5)
- added R14: 715k/0603/1%, Resistor_SMD:R_0603_1608Metric, F.Cu at (140.8, 53.5)
- added R44: 1M/0603/1%, Resistor_SMD:R_0603_1608Metric, F.Cu at (138.4, 52.7)
- C10, C11, C13, C18, C20, C9: value 120n/50V/0603 -> 100n/50V/0603
- C15: value 10u/50V/1206 -> 1uF/50V/1206
- C8: value 120n/50V/0603 -> 100nF/50V/0603
- J1: value 640388-3 -> 2157601003; footprint Library:TE_640388-3 -> Library:MOLEX_2157601003
- R10, R4, R9: value 1.8k/0603/1% -> 590R/0603/1%
- R11: value 1k/0603/1% -> 1.82k/0603/1%
- R5: value 2.05k/0603/1% -> 681R/0603/1%
- R6: value 6.19k/0603/1% -> 4.22k/0603/1%
- R7: value 2.43k/0603/1% -> 806R/0603/1%
- U10, U11, U12, U3, U4, U5, U8: value SIP32433ADN-T1E4 -> TPS259571DSGR; footprint Library:DFN-10-1EP_3x3mm_P0.5mm_EP1.7x2.5mm -> Library:SON50P200X200X80-9N
- moved R11 33.3 mm to (132.3, 97.1), turned to 180 degrees
- moved R7 7.47 mm to (110.8, 97.1), turned to 180 degrees
- moved R9 7.17 mm to (121.9, 97.1), turned to 180 degrees
- moved R5 7.11 mm to (144.0, 97.0), turned to 180 degrees
- moved R6 6.99 mm to (161.1, 80.2), turned to 180 degrees
- moved R10 6.71 mm to (110.8, 78.3), turned to 180 degrees
- moved R4 6.60 mm to (149.0, 68.1), turned to -90 degrees
- moved J1 4.63 mm to (124.3, 57.4)
- moved C13 2.08 mm to (107.4, 91.0)
- moved C15 2.08 mm to (149.1, 71.9)
- moved C27 2.03 mm to (128.2, 97.1)
- moved C7 2.02 mm to (128.2, 88.9)
- moved C17 2.01 mm to (106.5, 71.1)
- moved C12 1.99 mm to (106.6, 89.0)
- moved C14 1.98 mm to (117.8, 88.9)
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Connections:
- C10 pad 1: Net-(U5-SS) -> +12V
- C11 pad 1: Net-(U10-SS) -> +12V
- C13 pad 1: Net-(U8-SS) -> +5V
- C18 pad 1: Net-(U11-SS) -> +5V
- C20 pad 1: Net-(U12-SS) -> +5V
- C8 pad 1: Net-(U3-SS) -> +12V
- C9 pad 1: Net-(U4-SS) -> +12V
- R10 pad 2: Net-(U12-ILim) -> Net-(U12-ILM)
- R11 pad 2: Net-(U3-OVP) -> Net-(U5-ILM)
- R26 pad 1: +5V -> /V_EN
- R27 pad 1: +5V -> /V_EN
- R28 pad 1: +5V -> /V_EN
- R4 pad 2: Net-(U3-ILim) -> Net-(U3-ILM)
- R5 pad 2: Net-(U4-ILim) -> Net-(U4-ILM)
- R6 pad 2: Net-(U10-ILim) -> Net-(U10-ILM)
- R7 pad 2: Net-(U8-ILim) -> Net-(U8-ILM)
- R9 pad 2: Net-(U11-ILim) -> Net-(U11-ILM)
- U10 pad 1: +12V -> Net-(U10-DVDT)
- U10 pad 2: +12V -> /V_EN
- U10 pad 3: Net-(U10-SS) -> +12V
- U10 pad 4: Net-(U10-EN/UVLO) -> +12V
- U10 pad 5: Net-(U10-ILim) -> /+12V-0.2A
- U10 pad 6: GND -> unconnected-(U10-~{FLT}-Pad6)
- U10 pad 7: Net-(U10-OVP) -> Net-(U10-ILM)
- U10 pad 8: unconnected-(U10-PG-Pad8) -> GND
- U10 pad 9: /+12V-0.2A -> GND
- U11 pad 1: +5V -> Net-(U11-DVDT)
- U11 pad 3: Net-(U11-SS) -> +5V
- U11 pad 4: Net-(U11-EN/UVLO) -> +5V
- U11 pad 5: Net-(U11-ILim) -> /+5V-3A_1
- U11 pad 6: GND -> unconnected-(U11-~{FLT}-Pad6)
- U11 pad 7: Net-(U11-OVP) -> Net-(U11-ILM)
- U11 pad 8: unconnected-(U11-PG-Pad8) -> GND
- U11 pad 9: /+5V-3A_1 -> GND
- U12 pad 1: +5V -> Net-(U12-DVDT)
- U12 pad 3: Net-(U12-SS) -> +5V
- U12 pad 4: Net-(U12-EN/UVLO) -> +5V
- U12 pad 5: Net-(U12-ILim) -> /+5V-3A_2
- U12 pad 6: GND -> unconnected-(U12-~{FLT}-Pad6)
- U12 pad 7: Net-(U12-OVP) -> Net-(U12-ILM)
- U12 pad 8: unconnected-(U12-PG-Pad8) -> GND
- U12 pad 9: /+5V-3A_2 -> GND
- U3 pad 1: +12V -> Net-(U3-DVDT)
- U3 pad 2: +12V -> /V_EN
- U3 pad 3: Net-(U3-SS) -> +12V
- U3 pad 4: Net-(U3-EN/UVLO) -> +12V
- U3 pad 5: Net-(U3-ILim) -> /+12V-3A
- U3 pad 6: GND -> unconnected-(U3-~{FLT}-Pad6)
- U3 pad 7: Net-(U3-OVP) -> Net-(U3-ILM)
- U3 pad 8: unconnected-(U3-PG-Pad8) -> GND
- U3 pad 9: /+12V-3A -> GND
- U4 pad 1: +12V -> Net-(U4-DVDT)
- U4 pad 2: +12V -> /V_EN
- U4 pad 3: Net-(U4-SS) -> +12V
- U4 pad 4: Net-(U4-EN/UVLO) -> +12V
- U4 pad 5: Net-(U4-ILim) -> /+12V-2.5A
- U4 pad 6: GND -> unconnected-(U4-~{FLT}-Pad6)
- U4 pad 7: Net-(U4-OVP) -> Net-(U4-ILM)
- U4 pad 8: unconnected-(U4-PG-Pad8) -> GND
- U4 pad 9: /+12V-2.5A -> GND
- U5 pad 1: +12V -> Net-(U5-DVDT)
- U5 pad 2: +12V -> /V_EN
- U5 pad 3: Net-(U5-SS) -> +12V
- U5 pad 4: Net-(U5-EN/UVLO) -> +12V
- U5 pad 5: Net-(U5-ILim) -> /+12V-1A
- U5 pad 6: GND -> unconnected-(U5-~{FLT}-Pad6)
- U5 pad 7: Net-(U5-OVP) -> Net-(U5-ILM)
- U5 pad 8: unconnected-(U5-PG-Pad8) -> GND
- U5 pad 9: /+12V-1A -> GND
- U8 pad 1: +5V -> Net-(U8-DVDT)
- U8 pad 3: Net-(U8-SS) -> +5V
- U8 pad 4: Net-(U8-EN/UVLO) -> +5V
- U8 pad 5: Net-(U8-ILim) -> /+5V-2A
- U8 pad 6: GND -> unconnected-(U8-~{FLT}-Pad6)
- U8 pad 7: Net-(U8-OVP) -> Net-(U8-ILM)
- U8 pad 8: unconnected-(U8-PG-Pad8) -> GND
- U8 pad 9: /+5V-2A -> GND
