File: Connector_Extension_Board_V1.0/Connector_Extension_Board_V1.0.kicad_sch (KiCad schematic)
At the start: 75 parts, among them J1 640388-3, U10 SIP32433ADN-T1E4, U11 SIP32433ADN-T1E4, U12 SIP32433ADN-T1E4, U3 SIP32433ADN-T1E4, U4 SIP32433ADN-T1E4, U5 SIP32433ADN-T1E4, U8 SIP32433ADN-T1E4, U9 TPS1HC30BQPWPRQ1

Commit message: Hoan thanh chinh sua theo phan hoi 12/1
Parts:
- removed R12, R13, R16, R17, R19, R37: 1k/0603/1%, Resistor_SMD:R_0603_1608Metric, symbol Device:R
- removed R29, R31, R33, R35, R38, R40, R42: 100k/0603/1%, Resistor_SMD:R_0603_1608Metric, symbol Device:R
- removed R30, R32, R34, R36: 10.7k/0603/1%, Resistor_SMD:R_0603_1608Metric, symbol Device:R
- removed R39, R41, R43: 4.87k/0603/1%, Resistor_SMD:R_0603_1608Metric, symbol Device:R
- removed R8: 4.12k/0603/1%, Resistor_SMD:R_0603_1608Metric, symbol Device:R
- removed U10, U11, U12, U3, U4, U5, U8: SIP32433ADN-T1E4, Library:DFN-10-1EP_3x3mm_P0.5mm_EP1.7x2.5mm, symbol Library:SIP32433ADN-T1E4
- added C23, C24, C25, C29, C30, C31, C32: 3.3nF/50V/0603, Capacitor_SMD:C_0603_1608Metric, symbol Device:C
- added R14: 715k/0603/1%, Resistor_SMD:R_0603_1608Metric, symbol Device:R
- added R44: 1M/0603/1%, Resistor_SMD:R_0603_1608Metric, symbol Device:R
- added U10, U11, U12, U3, U4, U5, U8: TPS259571DSGR, Library:SON50P200X200X80-9N, symbol Library:TPS259571DSGR
- C10, C11, C13, C18, C20, C9: value 120n/50V/0603 -> 100n/50V/0603
- C15: value 10u/50V/1206 -> 1uF/50V/1206
- C8: value 120n/50V/0603 -> 100nF/50V/0603
- J1: value 640388-3 -> 2157601003; footprint Library:TE_640388-3 -> Library:MOLEX_2157601003; DIGIKEY (none) -> 900-2157601003-ND
- R10, R4, R9: value 1.8k/0603/1% -> 590R/0603/1%
- R11: value 1k/0603/1% -> 1.82k/0603/1%
- R26: now not fitted
- R5: value 2.05k/0603/1% -> 681R/0603/1%
- R6: value 6.19k/0603/1% -> 4.22k/0603/1%
- R7: value 2.43k/0603/1% -> 806R/0603/1%
Connections:
- net +12V: now also C10.1, C11.1, C8.1, C9.1, R44.2, U10.3 (IN), U10.4 (IN__1), U3.3 (IN), U3.4 (IN__1), U4.3 (IN), U4.4 (IN__1), U5.3 (IN), U5.4 (IN__1)
- net +12V-0.2A: now also U10.5 (OUT)
- net +12V-1A: now also U5.5 (OUT)
- net +12V-2.5A: now also U4.5 (OUT)
- net +12V-3A: now also U3.5 (OUT)
- net +5V: now also C13.1, C18.1, C20.1, U11.2 (EN/UVLO), U11.3 (IN), U11.4 (IN__1), U12.2 (EN/UVLO), U12.3 (IN), U12.4 (IN__1), U8.2 (EN/UVLO), U8.3 (IN), U8.4 (IN__1); no longer R26.1, R27.1, R28.1
- net +5V-2A: now also U8.5 (OUT)
- net +5V-3A_1: now also U11.5 (OUT)
- net +5V-3A_2: now also U12.5 (OUT)
- net GND: now also C23.2, C24.2, C25.2, C29.2, C30.2, C31.2, C32.2, R14.1, U10.8 (GND), U10.9 (GND__1), U11.8 (GND), U11.9 (GND__1), U12.8 (GND), U12.9 (GND__1), U3.8 (GND), U3.9 (GND__1), U4.8 (GND), U4.9 (GND__1), U5.8 (GND), U5.9 (GND__1), U8.8 (GND), U8.9 (GND__1)
- net at R9.2: now also U11.7 (ILM)
- net at R7.2: now also U8.7 (ILM)
- net at R5.2: now also U4.7 (ILM)
- net at R6.2: now also U10.7 (ILM)
- net at R10.2: now also U12.7 (ILM)
- net at R11.2: now also U5.7 (ILM)
- net at R4.2: now also U3.7 (ILM)
- new net: C24.1, U4.1 (DVDT)
- new net: C29.1, U10.1 (DVDT)
- new net: C31.1, U11.1 (DVDT)
- new net: C23.1, U3.1 (DVDT)
- new net: C25.1, U5.1 (DVDT)
- new net: C30.1, U8.1 (DVDT)
- new net: C32.1, U12.1 (DVDT)
- new net V_EN: R14.2, R26.1, R27.1, R28.1, R44.1, U10.2 (EN/UVLO), U3.2 (EN/UVLO), U4.2 (EN/UVLO), U5.2 (EN/UVLO)
Other:
- note added: "Auto-Retry Mode"
- note added: "Imax: 13A Pitch: 3mm"
- note added: "Rlim= 2000/(ILim -0.04) Ilim=0.51A Rlim=4220 ohm"
- note added: "Rlim= 2000/(ILim -0.04) Ilim=1.14A Rlim=1820 ohm"
- note added: "Rlim= 2000/(ILim -0.04) Ilim=2.5 Rlim=806 ohm"
- note added: "Rlim= 2000/(ILim -0.04) Ilim=2.97A Rlim=681 ohm"
- note added: "Rlim= 2000/(ILim -0.04) Ilim=3.43 Rlim=590 ohm"
- note added: "Since a 1% resistor is used, the E96 standard values are applied."
- note removed: "BACKup: 350790-1"
- note removed: "ILim=(0.6/RLim)*10300 0.99A"
- note removed: "ILim=(0.6/RLim)*10300 1.5A"
- note removed: "ILim=(0.6/RLim)*10300 2.54A"
- note removed: "ILim=(0.6/RLim)*10300 3.01A"
- note removed: "ILim=(0.6/RLim)*10300 3.43A"
- note removed: "Imax: 14.4A Pitch: 3.96mm"
- note removed: "OVP: 14.04V"
- note removed: "OVP: 7.04V"
- note removed: "Since a 1% resistor is used, the E92 standard values are applied."
- moved on the sheet: C15, C4, C8, Computer1, R10, R4, R5, R6, R7, R9
