File: Power_management_V2/5V.kicad_sch (KiCad schematic)
At the start: 29 parts, among them U5 SIC43x

Commit message: Hoan thanh SCH mach Power
Parts:
- removed C22, C23, C24: 22u, Library:C_CER_7.5x6.3, symbol Device:C
- removed C26, C29: 100n, Library:C_0603_1608Metric, symbol Device:C
- removed C30, C31, C32, C33, C34, C35, C36, C37, C38, C39, C40, C41: 22u, Library:C_1210_3225Metric, symbol Device:C
- removed R21: 100k, Library:R_0603_1608Metric, symbol Device:R
- added C1, C3, C4, C5, C6, C7, C8, C9: 22u/50V/3025, Library:C_CER_7.5x6.3, symbol Device:C
- added C10, C2: 100n/50V/0603, Library:C_0603_1608Metric, symbol Device:C
- added R1, R2: 100k/0603, Library:R_0603_1608Metric, symbol Device:R
- C21: value 22u -> 22u/50V/3025
- C25: value 100n -> 100n/50V/0603
- C27: value 4.7u -> 4.7u/16V/1206
- C28: value 1u -> 1u/16V/0603
- L5: value 2.2u -> 2.2u/22A; footprint Library:L_Vishay_IHLP-6767 -> (none); Current 16A -> (none); Digikey 541-1253-1-ND -> SRP1265A-2R2M; Isat 12 -> (none); Manufacturer VISHAY -> (none); Part IHLP6767GZER2R2M01 -> SRP1265A-2R2M; Resistance 2.4m -> (none)
- R19: value 2.2 -> 2.2R/0603
- R20: value 100k -> 100k/0603
- R22: value 100k -> 200k/0603; Digikey 13-RC0603FR-13200KLCT-ND -> (none); Manufacturer YAGEO -> (none); Part RC0603FR-13200KL -> (none); Power 1/10 -> (none); Tolerance 1% -> (none)
- R23: value 10k -> 10k/0603/0.1%
- R24: value 191K -> 73.2K/0603/0.1; Digikey A110327CT-ND -> (none); Manufacturer TE Connectivity Passive Product -> (none); Part 1-2176090-7 -> (none); Power 1/16 -> (none); Tolerance 0.1% -> (none)
Connections:
- net GND: now also C1.2, C10.1, C3.2, C4.2, C5.2, C6.2, C7.2, C8.2, C9.2
- net VBAT: now also C1.1, R2.1
- net VOUT: now also C10.2, C3.1, C4.1, C5.1, C6.1, C7.1, C8.1, C9.1
- net at C28.1, R20.2, U5.15 (VDD): now also R1.1
- net at U5.21 (MODE1): now also R1.2
- net at U5.23 (BOOT): now also C2.1
- net at R19.2: now also C2.2
- net EN: no longer names the net of U5.19 (EN)
- net EN: now also R2.2
- net P_GOOD: no longer names the net of R20.1, U5.14 (PGOOD)
Other:
- note added: "AGND and PGND connected inside SIC437"
- note added: "MODE selection MODE1 100K to VDD for forced CCM Fsw = 500kHz MODE2 OC limit of 14A 200K to AGND = 78% of Imax (18A - SIC437x)"
- note added: "Output Voltage ------- R_FB_H = R_FB_L(Vout-Vfb)/Vfb R_FB_H - Resistor Feedback High R_FB_L - Resistor feedback Low VOut - Desired output voltage Vfb - feedback voltage (0.6) ------ R_FB_H = 10000(5-0.6)/0.6 R_FB_H = 73.2k"
- note added: "SIC437AED-T1-GE3"
- note removed: "Output Voltage ------- R_FB_H = R_FB_L(Vout-Vfb)/Vfb R_FB_H - Resistor Feedback High R_FB_L - Resistor feedback Low VOut - Desired output voltage Vfb - feedback voltage (0.6) ------ R_FB_H = 10000(12-0.6)/0.6 R_FB_H = 190k"
- moved on the sheet: C25

Commit message: Hoan thanh SCH lan 1
Parts:
- removed R24: 73.2K/0603/0.1, Library:R_0603_1608Metric, symbol Device:R
- added R14: 73.2K/0603/0.1, Library:R_0603_1608Metric, symbol Device:R
- renumbered C21 to C20, C1 to C21, C25 to C22, C2 to C23, C27 to C24, C28 to C25, C10 to C26, C3 to C27, C4 to C28, C5 to C29, C6 to C30, C7 to C31, C8 to C32, C9 to C33, L5 to L2, R22 to R10, R20 to R11, R1 to R12, R23 to R13, R2 to R8, R19 to R9, U5 to U2
Connections:
- net VOUT: now also R14.2
- net at R13.2, U2.17 (FB): now also R14.1

Commit message: Chỉnh sủa SCH 24/12
Parts:
- removed R8: 100k/0603, Library:R_0603_1608Metric, symbol Device:R
Connections:
- net EN_5V: now reaches U2.19 (EN)
- now unconnected: U2.10 (GL), U2.11 (GL), U2.28 (GL)
- no-connect marks 0 -> 3
Other:
- company: Raw Matter IO Pty Ltd -> (none)
- title: (none) -> Diptek Power Board V2
Changed lines of the file:
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@@
 	(paper "A4")
 	(title_block
+		(title "Diptek Power Board V2")
 		(date "2025-08-26")
-		(rev "1")
-		(company "Raw Matter IO Pty Ltd")
-		(comment 1 "Preliminary Design")
-		(comment 2 "Released for discussion")
-		(comment 3 "C28 updated")
+		(rev "2")
 	)
 	(text "Output Voltage\n-------\nR_FB_H = R_FB_L(Vout-Vfb)/Vfb\nR_FB_H - Resistor Feedback High\nR_FB_L - Resistor feedback Low\nVOut - Desired output voltage\nVfb - feedback voltage (0.6)\n------\nR_FB_H = 10000(5-0.6)/0.6\nR_FB_H = 73.2k\n"
@@
 	)
 	(junction
-		(at 106.045 68.58)
-		(diameter 0)
-		(color 0 0 0 0)
-	)
-	(junction
 		(at 259.08 106.68)
 		(diameter 0)
@@
 	)
 	(junction
+		(at 190.5 106.68)
+		(diameter 0)
+		(color 0 0 0 0)
+	)
+	(no_connect
+		(at 137.16 95.25)
+	)
+	(no_connect
+		(at 137.16 100.33)
+	)
+	(no_connect
 		(at 137.16 97.79)
-		(diameter 0)
-		(color 0 0 0 0)
-	)
-	(junction
-		(at 190.5 106.68)
-		(diameter 0)
-		(color 0 0 0 0)
 	)
 	(wire
@@
 	(wire
 		(pts
-			(xy 118.745 76.2) (xy 139.7 76.2)
+			(xy 113.03 76.2) (xy 139.7 76.2)
 		)
 		(stroke
@@
 	(wire
 		(pts
-			(xy 111.125 76.2) (xy 106.045 76.2)
-		)
-		(stroke
-			(width 0)
-			(type default)
-		)
-	)
-	(wire
-		(pts
 			(xy 161.29 85.09) (xy 167.64 85.09)
 		)
@@
 	(wire
 		(pts
-			(xy 91.44 68.58) (xy 106.045 68.58)
-		)
-		(stroke
-			(width 0)
-			(type default)
-		)
-	)
-	(wire
-		(pts
 			(xy 179.07 72.39) (xy 168.91 72.39)
 		)
@@
 	(wire
 		(pts
-			(xy 137.16 97.79) (xy 137.16 100.33)
-		)
-		(stroke
-			(width 0)
-			(type default)
-		)
-	)
-	(wire
-		(pts
-			(xy 137.16 95.25) (xy 137.16 97.79)
-		)
-		(stroke
-			(width 0)
-			(type default)
-		)
-	)
-	(wire
-		(pts
 			(xy 72.39 76.2) (xy 81.28 76.2)
 		)
@@
 	(wire
 		(pts
-			(xy 106.045 76.2) (xy 106.045 68.58)
-		)
-		(stroke
-			(width 0)
-			(type default)
-		)
-	)
-	(wire
-		(pts
 			(xy 161.29 111.76) (xy 163.83 111.76)
 		)
@@
 	(wire
 		(pts
-			(xy 106.045 68.58) (xy 139.7 68.58)
+			(xy 91.44 68.58) (xy 139.7 68.58)
 		)
 		(stroke
@@
 			(width 0)
 			(type default)
+		)
+	)
+	(hierarchical_label "EN_5V"
+		(shape input)
+		(at 113.03 76.2 180)
+		(effects
+			(font
+				(size 1.27 1.27)
+			)
+			(justify right)
 		)
 	)
@@
 					(unit 1)
 				)
-			)
-		)
-	)
-	(symbol
-		(lib_id "Device:R")
-		(at 114.935 76.2 90)
-		(unit 1)
-		(exclude_from_sim no)
-		(in_bom yes)
-		(on_board yes)
-		(dnp no)
-		(fields_autoplaced yes)
-		(property "Reference" "R8"
-			(at 114.935 70.485 90)
-			(effects
-				(font
-					(size 1.27 1.27)
-				)
-			)
-		)
-		(property "Value" "100k/0603"
-			(at 114.935 73.025 90)
-			(effects
-				(font
-					(size 1.27 1.27)
-				)
-			)
-		)
-		(property "Footprint" "Library:R_0603_1608Metric"
-			(at 114.935 77.978 90)
-			(effects
-				(font
-					(size 1.27 1.27)
-				)
-				(hide yes)
-			)
-		)
-		(property "Datasheet" ""
-			(at 114.935 76.2 0)
-			(effects
-				(font
-					(size 1.27 1.27)
-				)
-				(hide yes)
-			)
-		)
-		(property "Description" "Resistor"
-			(at 114.935 76.2 0)
-			(effects
-				(font
-					(size 1.27 1.27)
-				)
-				(hide yes)
-			)
-		)
-		(property "Digikey" "311-100KHRCT-ND"
-			(at 114.935 76.2 0)
-			(effects
-				(font
-					(size 1.27 1.27)
-				)
-				(hide yes)
-			)
-		)
-		(property "Power" "1/16"
-			(at 114.935 76.2 0)
-			(effects
-				(font
-					(size 1.27 1.27)
-				)
-				(hide yes)
-			)
-		)
-		(property "Tolerance" "1%"
-			(at 114.935 76.2 0)
-			(effects
-				(font
-					(size 1.27 1.27)
-				)
-				(hide yes)
-			)
-		)
-		(property "Manufacturer" "YAGEO"
-			(at 114.935 76.2 0)
-			(effects
-				(font
-					(size 1.27 1.27)
-				)
-				(hide yes)
-			)
-		)
-		(property "Part" "RC0603FR-07100KL"
-			(at 114.935 76.2 0)
-			(effects
-				(font
-					(size 1.27 1.27)
-				)
-				(hide yes)
-			)
-		)
-		(pin "1"
-		)
-		(pin "2"
-		)
-		(instances
-			(project "Power_management_V2"
-				(path "/632966f8-0e72-49d8-ae31-468f807051b0/72d31167-e5b9-4ad1-a5a3-7c9d97c1c508"
-					(reference "R8")
-					(unit 1)
-				)

Commit message: Hoan thanh footprint
Parts:
- C22, C23, C25, C26: footprint Library:C_0603_1608Metric -> Capacitor_SMD:C_0603_1608Metric
- L2: footprint (none) -> Library:IND_SRP1265A-2R2M
- R10, R11, R12, R13, R14, R9: footprint Library:R_0603_1608Metric -> Resistor_SMD:R_0603_1608Metric
- U2: footprint Library:SIC43x -> Library:VREG_SIC437AED-T1-GE3

Commit message: hoan thanh sap xep
Parts:
- C27, C28, C29, C30, C31, C32, C33: value 22u/50V/3025 -> 22u/25V/1210; footprint Library:C_CER_7.5x6.3 -> Capacitor_SMD:C_1210_3225Metric
Changed lines of the file:
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@@
 			)
 		)
-		(property "Value" "22u/50V/3025"
+		(property "Value" "22u/25V/1210"
 			(at 208.28 130.175 90)
 			(effects
@@
 			)
 		)
-		(property "Footprint" "Library:C_CER_7.5x6.3"
+		(property "Footprint" "Capacitor_SMD:C_1210_3225Metric"
 			(at 211.7852 114.3 0)
 			(effects
@@
 			)
 		)
-		(property "Value" "22u/50V/3025"
+		(property "Value" "22u/25V/1210"
 			(at 245.11 125.095 90)
 			(effects
@@
 			)
 		)
-		(property "Footprint" "Library:C_CER_7.5x6.3"
+		(property "Footprint" "Capacitor_SMD:C_1210_3225Metric"
 			(at 250.5202 114.3 0)
 			(effects
@@
 			)
 		)
-		(property "Value" "22u/50V/3025"
+		(property "Value" "22u/25V/1210"
 			(at 216.535 125.095 90)
 			(effects
@@
 			)
 		)
-		(property "Footprint" "Library:C_CER_7.5x6.3"
+		(property "Footprint" "Capacitor_SMD:C_1210_3225Metric"
 			(at 221.9452 114.3 0)
 			(effects
@@
 			)
 		)
-		(property "Value" "22u/50V/3025"
+		(property "Value" "22u/25V/1210"
 			(at 254.635 125.095 90)
 			(effects
@@
 			)
 		)
-		(property "Footprint" "Library:C_CER_7.5x6.3"
+		(property "Footprint" "Capacitor_SMD:C_1210_3225Metric"
 			(at 260.0452 114.3 0)
 			(effects
@@
 			)
 		)
-		(property "Value" "22u/50V/3025"
+		(property "Value" "22u/25V/1210"
 			(at 235.585 125.095 90)
 			(effects
@@
 			)
 		)
-		(property "Footprint" "Library:C_CER_7.5x6.3"
+		(property "Footprint" "Capacitor_SMD:C_1210_3225Metric"
 			(at 240.9952 114.3 0)
 			(effects
@@
 			)
 		)
-		(property "Value" "22u/50V/3025"
+		(property "Value" "22u/25V/1210"
 			(at 264.16 125.095 90)
 			(effects
@@
 			)
 		)
-		(property "Footprint" "Library:C_CER_7.5x6.3"
+		(property "Footprint" "Capacitor_SMD:C_1210_3225Metric"
 			(at 269.5702 114.3 0)
 			(effects
@@
 			)
 		)
-		(property "Value" "22u/50V/3025"
+		(property "Value" "22u/25V/1210"
 			(at 226.06 125.095 90)
 			(effects
@@
 			)
 		)
-		(property "Footprint" "Library:C_CER_7.5x6.3"
+		(property "Footprint" "Capacitor_SMD:C_1210_3225Metric"
 			(at 231.4702 114.3 0)
 			(effects

Commit message: Layout 2201
Parts:
- added NT1: NetTie_2, Library:NetTie-2_SMD_Pad1.56mm, symbol Device:NetTie_2
Connections:
- net GND: now also C24.2, NT1.2
- net GND1: now also NT1.1; no longer C24.2
Changed lines of the file:
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@@
 	(wire
 		(pts
+			(xy 156.21 127.635) (xy 156.21 124.46)
+		)
+		(stroke
+			(width 0)
+			(type default)
+		)
+	)
+	(wire
+		(pts
 			(xy 161.29 109.22) (xy 190.5 109.22)
 		)
@@
 	(wire
 		(pts
+			(xy 151.13 124.46) (xy 151.13 127.635)
+		)
+		(stroke
+			(width 0)
+			(type default)
+		)
+	)
+	(wire
+		(pts
 			(xy 134.62 90.17) (xy 139.7 90.17)
 		)
@@
 	(symbol
 		(lib_id "power:GND")
+		(at 163.83 119.38 0)
+		(unit 1)
+		(exclude_from_sim no)
+		(in_bom yes)
+		(on_board yes)
+		(dnp no)
+		(fields_autoplaced yes)
+		(property "Reference" "#PWR021"
+			(at 163.83 125.73 0)
+			(effects
+				(font
+					(size 1.27 1.27)
+				)
+				(hide yes)
+			)
+		)
+		(property "Value" "GND"
+			(at 163.83 123.8234 0)
+			(effects
+				(font
+					(size 1.27 1.27)
+				)
+			)
+		)
+		(property "Footprint" ""
+			(at 163.83 119.38 0)
+			(effects
+				(font
+					(size 1.27 1.27)
+				)
+				(hide yes)
+			)
+		)
+		(property "Datasheet" ""
+			(at 163.83 119.38 0)
+			(effects
+				(font
+					(size 1.27 1.27)
+				)
+				(hide yes)
+			)
+		)
+		(property "Description" ""
+			(at 163.83 119.38 0)
+			(effects
+				(font
+					(size 1.27 1.27)
+				)
+			)
+		)
+		(pin "1"
+		)
+		(instances
+			(project "Power_management_V2"
+				(path "/632966f8-0e72-49d8-ae31-468f807051b0/72d31167-e5b9-4ad1-a5a3-7c9d97c1c508"
+					(reference "#PWR021")
+					(unit 1)
+				)
+			)
+		)
+	)
+	(symbol
+		(lib_id "power:GND")
 		(at 230.505 114.3 0)
 		(unit 1)
@@
 	)
 	(symbol
+		(lib_id "power:GND")
+		(at 151.13 127.635 0)
+		(unit 1)
+		(exclude_from_sim no)
+		(in_bom yes)
+		(on_board yes)
+		(dnp no)
+		(fields_autoplaced yes)
+		(property "Reference" "#PWR022"
+			(at 151.13 133.985 0)
+			(effects
+				(font
+					(size 1.27 1.27)
+				)
+				(hide yes)
+			)
+		)
+		(property "Value" "GND"
+			(at 151.13 132.0784 0)
+			(effects
+				(font
+					(size 1.27 1.27)
+				)
+			)
+		)
+		(property "Footprint" ""
+			(at 151.13 127.635 0)
+			(effects
+				(font
+					(size 1.27 1.27)
+				)
+				(hide yes)
+			)
+		)
+		(property "Datasheet" ""
+			(at 151.13 127.635 0)
+			(effects
+				(font
+					(size 1.27 1.27)
+				)
+				(hide yes)
+			)
+		)
+		(property "Description" ""
+			(at 151.13 127.635 0)
+			(effects
+				(font
+					(size 1.27 1.27)
+				)
+			)
+		)
+		(pin "1"
+		)
+		(instances
+			(project "Power_management_V2"
+				(path "/632966f8-0e72-49d8-ae31-468f807051b0/72d31167-e5b9-4ad1-a5a3-7c9d97c1c508"
+					(reference "#PWR022")
+					(unit 1)
+				)
+			)
+		)
+	)
+	(symbol
 		(lib_id "Device:C")
 		(at 91.44 72.39 180)
@@
 	)
 	(symbol
-		(lib_id "power:GND1")
-		(at 163.83 119.38 0)
+		(lib_id "Device:NetTie_2")
+		(at 153.67 124.46 180)
 		(unit 1)
 		(exclude_from_sim no)
-		(in_bom yes)
+		(in_bom no)
 		(on_board yes)
 		(dnp no)
 		(fields_autoplaced yes)
-		(property "Reference" "#PWR014"
-			(at 163.83 125.73 0)
+		(property "Reference" "NT1"
+			(at 153.67 119.38 0)
 			(effects
 				(font
 					(size 1.27 1.27)
 				)
-				(hide yes)
 			)
 		)
-		(property "Value" "GND1"
-			(at 163.83 124.46 0)
+		(property "Value" "NetTie_2"
+			(at 153.67 121.92 0)
 			(effects
 				(font
@@
 			)
 		)
-		(property "Footprint" ""
-			(at 163.83 119.38 0)
+		(property "Footprint" "Library:NetTie-2_SMD_Pad1.56mm"
+			(at 153.67 124.46 0)
 			(effects
 				(font
@@
 			)
 		)
-		(property "Datasheet" ""
-			(at 163.83 119.38 0)
+		(property "Datasheet" "~"
+			(at 153.67 124.46 0)
 			(effects
 				(font
@@
 			)
 		)
-		(property "Description" ""
-			(at 163.83 119.38 0)
+		(property "Description" "Net tie, 2 pins"
+			(at 153.67 124.46 0)
 			(effects
 				(font
 					(size 1.27 1.27)
 				)
+				(hide yes)
 			)
 		)
+		(pin "2"
+		)
 		(pin "1"
 		)
 		(instances
-			(project "Power_management_V2"
+			(project ""
 				(path "/632966f8-0e72-49d8-ae31-468f807051b0/72d31167-e5b9-4ad1-a5a3-7c9d97c1c508"
-					(reference "#PWR014")
+					(reference "NT1")
 					(unit 1)
 				)
@@
 					(unit 1)
 				)
+			)
+		)
+	)
+	(symbol
+		(lib_id "power:GND1")
+		(at 156.21 127.635 0)
+		(unit 1)
+		(exclude_from_sim no)
+		(in_bom yes)
+		(on_board yes)
+		(dnp no)
+		(fields_autoplaced yes)
+		(property "Reference" "#PWR023"
+			(at 156.21 133.985 0)
+			(effects
+				(font
+					(size 1.27 1.27)
+				)
+				(hide yes)
+			)
+		)
+		(property "Value" "GND1"
+			(at 156.21 132.715 0)
+			(effects
+				(font
+					(size 1.27 1.27)
+				)
+			)
+		)
+		(property "Footprint" ""
+			(at 156.21 127.635 0)
+			(effects
+				(font
+					(size 1.27 1.27)
+				)
+				(hide yes)
+			)
+		)
+		(property "Datasheet" ""
+			(at 156.21 127.635 0)
+			(effects
+				(font
+					(size 1.27 1.27)
+				)
+				(hide yes)
+			)
+		)
+		(property "Description" ""
+			(at 156.21 127.635 0)
+			(effects
+				(font
+					(size 1.27 1.27)
+				)
+			)
+		)
+		(pin "1"
+		)
+		(instances
+			(project "Power_management_V2"
+				(path "/632966f8-0e72-49d8-ae31-468f807051b0/72d31167-e5b9-4ad1-a5a3-7c9d97c1c508"
+					(reference "#PWR023")
+					(unit 1)
+				)
