File: Power_management_V2/Power_management_V2.kicad_pcb (KiCad board)
At the start: 4 copper layers, 67.7 x 69 mm, 11 parts

Commit message: Hoan thanh footprint
Parts:
- removed 12V, 5V, GND: TestPoint_THTPad_3.0x3.0mm_Drill1.5mm, TestPoint:TestPoint_THTPad_3.0x3.0mm_Drill1.5mm
- removed Compute1, GPS1, Phone1: Conn_01x02, Library:TE_5-104809-1
- removed Winch1, Winch2, Winch3, Winch4, Winch5: Conn_01x02, Library:MOLEX_1722871102
- added BAT1: Conn_01x02, Library:Milwaukee 18V battery connector R1, F.Cu at (120.6, 72.2)
- added C1: 22u/50V/3025, Library:C_CER_7.5x6.3, F.Cu at (2.31, 10.2)
- added C10: 22u/50V/3025, Library:C_CER_7.5x6.3, F.Cu at (2.31, 36.8)
- added C11: 22u/50V/3025, Library:C_CER_7.5x6.3, F.Cu at (2.31, 45.6)
- added C12: 22u/50V/3025, Library:C_CER_7.5x6.3, F.Cu at (13.8, 10.2)
- added C13: 22u/50V/3025, Library:C_CER_7.5x6.3, F.Cu at (13.8, 19.1)
- added C14: 22u/50V/3025, Library:C_CER_7.5x6.3, F.Cu at (13.8, 27.9)
- added C15: 22u/50V/3025, Library:C_CER_7.5x6.3, F.Cu at (13.8, 36.8)
- added C16: 22u/50V/3025, Library:C_CER_7.5x6.3, F.Cu at (13.8, 45.6)
- added C17: 22u/50V/3025, Library:C_CER_7.5x6.3, F.Cu at (25.2, 10.2)
- added C18: 22u/50V/3025, Library:C_CER_7.5x6.3, F.Cu at (25.2, 19.1)
- added C19: 22u/50V/3025, Library:C_CER_7.5x6.3, F.Cu at (25.2, 27.9)
- added C2: 22u/50V/3025, Library:C_CER_7.5x6.3, F.Cu at (2.31, 19.1)
- added C20: 22u/50V/3025, Library:C_CER_7.5x6.3, F.Cu at (41.4, 56.5)
- added C21: 22u/50V/3025, Library:C_CER_7.5x6.3, F.Cu at (41.4, 65.3)
- added C22: 100n/50V/0603, Capacitor_SMD:C_0603_1608Metric, F.Cu at (53.4, 79.9)
- added C23: 100n/50V/0603, Capacitor_SMD:C_0603_1608Metric, F.Cu at (53.4, 82.4)
- added C24: 4.7u/16V/1206, Library:C_1206_3216Metric, F.Cu at (62.3, 86.4)
- added C25: 1u/16V/0603, Capacitor_SMD:C_0603_1608Metric, F.Cu at (53.4, 84.9)
- added C26: 100n/50V/0603, Capacitor_SMD:C_0603_1608Metric, F.Cu at (53.4, 87.4)
- added C27: 22u/50V/3025, Library:C_CER_7.5x6.3, F.Cu at (41.4, 74.2)
- added C28: 22u/50V/3025, Library:C_CER_7.5x6.3, F.Cu at (52.9, 56.5)
- added C29: 22u/50V/3025, Library:C_CER_7.5x6.3, F.Cu at (52.9, 65.3)
- added C3: 100n/50V/0603, Capacitor_SMD:C_0603_1608Metric, F.Cu at (32.9, 21.1)
- added C30: 22u/50V/3025, Library:C_CER_7.5x6.3, F.Cu at (52.9, 74.2)
- added C31: 22u/50V/3025, Library:C_CER_7.5x6.3, F.Cu at (64.3, 56.5)
- added C32: 22u/50V/3025, Library:C_CER_7.5x6.3, F.Cu at (64.3, 65.3)
- added C33: 22u/50V/3025, Library:C_CER_7.5x6.3, F.Cu at (64.3, 74.2)
- added C34: 100n/50V/0603, Capacitor_SMD:C_0603_1608Metric, F.Cu at (12.6, 84.3)
- added C4: 100n/50V/0603, Capacitor_SMD:C_0603_1608Metric, F.Cu at (32.9, 23.6)
- added C5: 100n/50V/0603, Capacitor_SMD:C_0603_1608Metric, F.Cu at (32.9, 26.1)
- added C6: 4.7u/16V/1206, Library:C_1206_3216Metric, F.Cu at (41.8, 27.7)
- added C7: 1u/16V/0603, Capacitor_SMD:C_0603_1608Metric, F.Cu at (32.9, 28.7)
- added C8: 100n/50V/0603, Capacitor_SMD:C_0603_1608Metric, F.Cu at (32.9, 31.2)
- added C9: 22u/50V/3025, Library:C_CER_7.5x6.3, F.Cu at (2.31, 27.9)
- added J1: 640388-3, Library:TE_640388-3, F.Cu at (139.1, 98.2)
- added L1: 2.2u/22A, Library:IND_SRP1265A-2R2M, F.Cu at (106.6, 93.7)
- added L2: 2.2u/22A, Library:IND_SRP1265A-2R2M, F.Cu at (125.6, 93.7)
- added R10: 200k/0603, Resistor_SMD:R_0603_1608Metric, F.Cu at (57.4, 79.9)
- added R11: 100k/0603, Resistor_SMD:R_0603_1608Metric, F.Cu at (57.4, 82.4)
- added R12: 100k/0603, Resistor_SMD:R_0603_1608Metric, F.Cu at (57.4, 84.9)
- added R13: 10k/0603/0.1%, Resistor_SMD:R_0603_1608Metric, F.Cu at (57.4, 87.4)
- added R14: 73.2K/0603/0.1, Resistor_SMD:R_0603_1608Metric, F.Cu at (57.4, 89.9)
- added R15: 2M/0603, Resistor_SMD:R_0603_1608Metric, F.Cu at (12.6, 89.3)
- added R16: 51.1K/0603, Resistor_SMD:R_0603_1608Metric, F.Cu at (12.6, 91.8)
- added R2: 2.2R/0603, Resistor_SMD:R_0603_1608Metric, F.Cu at (32.9, 33.7)
- added R3: 499k/0603, Resistor_SMD:R_0603_1608Metric, F.Cu at (37.0, 21.1)
- added R4: 100k/0603, Resistor_SMD:R_0603_1608Metric, F.Cu at (37.0, 23.6)
- added R5: 100k/0603, Resistor_SMD:R_0603_1608Metric, F.Cu at (37.0, 26.1)
- added R6: 10k/0603/0.1%, Resistor_SMD:R_0603_1608Metric, F.Cu at (37.0, 28.7)
- added R7: 191K/0603/0.1%, Resistor_SMD:R_0603_1608Metric, F.Cu at (37.0, 31.2)
- added R8: 100k/0603, Resistor_SMD:R_0603_1608Metric, F.Cu at (12.6, 86.8)
- added R9: 2.2R/0603, Resistor_SMD:R_0603_1608Metric, F.Cu at (53.4, 89.9)
- added U1: SIC43x, Library:VREG_SIC437AED-T1-GE3, F.Cu at (105.5, 79.3)
- added U2: SIC43x, Library:VREG_SIC437AED-T1-GE3, F.Cu at (112.0, 80.3)
- added U3: TPS3711DDCR, Package_TO_SOT_SMD:TSOT-23-6, F.Cu at (17.2, 85.5)
Routing:
- net (no net): vias 3 -> 0
Other:
- board size 67.7 x 69 mm -> 76.5 x 63 mm
- board text removed: "Compute1"
- board text removed: "Encoder"
- board text removed: "GPS1"
- board text removed: "LIDAR1"
- board text removed: "LoRa"
- board text removed: "Phone1"
- board text removed: "Spare"
- board text removed: "Winch1"

Commit message: hoan thanh sap xep
Parts:
- C10, C11, C12, C13, C14, C15, C16, C17, C18, C19, C27, C28, C29, C30, C31, C32, C33, C9: value 22u/50V/3025 -> 22u/25V/1210; footprint Library:C_CER_7.5x6.3 -> Capacitor_SMD:C_1210_3225Metric
- moved C13 162.3 mm to (161.9, 85.5)
- moved C14 162.3 mm to (161.9, 94.4)
- moved C15 162.3 mm to (161.9, 103.2)
- moved C9 139.6 mm to (117.6, 106.7), turned to -90 degrees
- moved C12 139.3 mm to (114.2, 106.8), turned to -90 degrees
- moved C34 133.7 mm to (144.7, 63.8), turned to -90 degrees
- moved C11 133.4 mm to (120.9, 106.7), turned to -90 degrees
- moved R16 132.5 mm to (142.7, 66.9), turned to 180 degrees
- moved R8 131.1 mm to (141.2, 61.3)
- moved R15 129.6 mm to (140.3, 67.7), turned to -90 degrees
- moved C1 128.8 mm to (121.5, 59.0)
- moved C2 128.5 mm to (121.5, 67.0)
- moved C10 126.7 mm to (109.0, 105.0), turned to -90 degrees
- moved U3 126.4 mm to (141.7, 64.0)
- moved C16 126.2 mm to (124.2, 106.7), turned to -90 degrees
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Other:
- board text added: "5V 12V GND"

Commit message: Hoan thien Sap xep Linh kien
Parts:
- removed C13: 22u/25V/1210, Capacitor_SMD:C_1210_3225Metric
- moved C27 44.5 mm to (118.0, 65.1), turned to -90 degrees
- moved C26 43.8 mm to (134.0, 58.4), turned to -90 degrees
- moved C33 41.9 mm to (131.6, 58.6), turned to 90 degrees
- moved C20 41.7 mm to (102.5, 100.6), turned to -90 degrees
- moved R14 41.5 mm to (92.2, 59.0), turned to -90 degrees
- moved C31 41.1 mm to (124.7, 58.5), turned to 90 degrees
- moved R13 41.1 mm to (94.5, 58.3), turned to 180 degrees
- moved C32 41.0 mm to (128.1, 58.6), turned to 90 degrees
- moved C24 39.7 mm to (99.0, 57.9), turned to 90 degrees
- moved C25 39.4 mm to (96.9, 58.7), turned to 90 degrees
- moved C30 38.8 mm to (121.5, 65.1), turned to -90 degrees
- moved C14 38.4 mm to (124.8, 104.2), turned to -90 degrees
- moved C21 36.1 mm to (110.5, 100.6), turned to -90 degrees
- moved C28 34.8 mm to (117.9, 58.6)
- moved C29 34.8 mm to (121.3, 58.6)
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
Commit message: Hoan thanh chinh sua theo phan hoi 12/1
Parts:
- removed C11: 22u/25V/1210, Capacitor_SMD:C_1210_3225Metric
- removed R3: 499k/0603, Resistor_SMD:R_0603_1608Metric
- added C13: 22u/25V/1210, Capacitor_SMD:C_1210_3225Metric, F.Cu at (125.4, 96.1)
- added C35: 22u/25V/1210, Capacitor_SMD:C_1210_3225Metric, F.Cu at (137.0, 84.1)
- added C36: 22u/25V/1210, Capacitor_SMD:C_1210_3225Metric, F.Cu at (119.1, 102.7)
- added R17: 200k/0603, Resistor_SMD:R_0603_1608Metric, F.Cu at (100.3, 86.9)
- J1: value 640388-3 -> 2165711003; footprint Library:TE_640388-3 -> Library:MOLEX_2165711003
- moved C15 7.93 mm to (125.3, 99.4), turned to 0 degrees
- moved J1 7.29 mm to (138.5, 90.9)
- moved C10 3.10 mm to (125.3, 102.9), turned to 0 degrees
- moved C14 2.18 mm to (125.3, 106.3), turned to 0 degrees
- moved C16 0.12 mm to (119.1, 106.1)

Commit message: Thay doi kich thuoc mach power
Parts:
- moved C20 5.16 mm to (97.5, 102.0)
- moved C21 5.16 mm to (105.5, 102.0)
- moved C2 4.91 mm to (96.8, 73.2)
- moved J1 3.58 mm to (140.1, 94.1)
- moved C22 3.16 mm to (95.1, 65.1)
- moved R11 3.16 mm to (92.8, 65.9)
- moved R9 3.16 mm to (90.5, 63.5)
- moved R10 3.16 mm to (89.7, 65.9)
- moved C23 3.16 mm to (90.5, 62.0)
- moved C25 3.16 mm to (94.8, 56.3)
- moved R13 3.16 mm to (92.5, 55.9)
- moved R14 3.16 mm to (90.1, 56.6)
- moved U2 3.16 mm to (95.2, 61.1)
- moved C24 3.16 mm to (96.9, 55.5)
- moved R12 3.16 mm to (91.3, 65.9)
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Other:
- board size 76.5 x 63 mm -> 76.5 x 66 mm

Commit message: Layout 2201
Parts:
- removed C3: 100n/50V/0603, Capacitor_SMD:C_0603_1608Metric
- added NT1: NetTie_2, Library:NetTie-2_SMD_Pad1.56mm, F.Cu at (95.1, 60.6)
- added NT2: NetTie_2, Library:NetTie-2_SMD_Pad1.56mm, F.Cu at (102.5, 88.1)
- moved R4 13.2 mm to (94.9, 81.3), turned to 180 degrees
- moved R11 11.9 mm to (87.2, 55.3), turned to 180 degrees
- moved C8 11.4 mm to (127.4, 94.9), turned to 180 degrees
- moved R5 10.3 mm to (94.2, 84.2), turned to -90 degrees
- moved R12 9.08 mm to (86.5, 58.1), turned to -90 degrees
- moved R10 7.92 mm to (88.0, 58.1), turned to 90 degrees
- moved C20 6.33 mm to (103.0, 105.1), turned to 0 degrees
- moved C21 5.45 mm to (103.0, 97.2), turned to 0 degrees
- moved R17 4.10 mm to (95.7, 84.2), turned to 90 degrees
- moved L1 2.76 mm to (116.0, 88.3)
- moved C27 1.49 mm to (119.0, 62.8)
- moved C31 1.49 mm to (125.7, 56.3)
- moved C33 1.49 mm to (132.6, 56.3)
- moved C28 1.49 mm to (118.9, 56.3)
- moved C29 1.49 mm to (122.3, 56.4)
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Connections:
- C24 pad 2: GND1 -> GND
- C6 pad 2: GND1 -> GND
- C7 pad 2: GND1 -> GND2
- R17 pad 2: GND1 -> GND2
- R6 pad 1: GND1 -> GND2
- U1 pad 16: GND1 -> GND2
- U1 pad 25: GND1 -> GND2
Routing:
- net /12V/EN_12V: track 0.00 -> 123.7 mm, vias 0 -> 6
- net /+5V: track 0.00 -> 35.8 mm, vias 0 -> 3
- net GND: track 0.00 -> 15.0 mm, vias 0 -> 5
- net Net-(U1-VDD): track 0.00 -> 14.7 mm, vias 0 -> 2
- net Net-(U2-VDD): track 0.00 -> 13.9 mm, vias 0 -> 2
- net Net-(U2-PGOOD): track 0.00 -> 13.2 mm
- net +BATT: track 0.00 -> 10.9 mm, vias 0 -> 4
- net GND1: track 0.00 -> 8.20 mm, vias 0 -> 4
- net Net-(U2-MODE1): track 0.00 -> 7.99 mm
- net Net-(U1-MODE1): track 0.00 -> 7.90 mm
- net Net-(U1-FB): track 0.00 -> 7.75 mm
- net Net-(U2-FB): track 0.00 -> 7.21 mm
- net Net-(U1-MODE2): track 0.00 -> 6.57 mm
- net Net-(U2-MODE2): track 0.00 -> 6.27 mm
- net Net-(U2-VDRV): track 0.00 -> 6.25 mm
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- added copper zone on F.Cu, net +BATT
- added copper zone on F.Cu, net /+12V
- added copper zone on F.Cu, net /+5V
- added copper zone on F.Cu, net Net-(L1-Pad1)
- added copper zone on F.Cu, net Net-(L2-Pad1)

Commit message: Hoan thanh layout PCB Power
Parts:
- moved C6 0.53 mm to (105.7, 83.6)
Routing:
- net /+12V: track 5.40 -> 34.1 mm
- net Net-(U1-PGOOD): track 0.00 -> 13.7 mm
- net GND: track 15.0 -> 20.8 mm, vias 5 -> 136
- net GND2: track 5.10 -> 9.97 mm, vias 2 -> 10
- net /12V/EN_12V: track 123.7 -> 118.8 mm
- net +BATT: track 10.9 -> 12.1 mm, vias 4 -> 97
- net /+5V: track 35.8 -> 35.6 mm, vias 3 -> 57
- net GND1: vias 4 -> 18
- net (no net): vias 90 -> 0
- added copper zone on B.Cu, net +BATT
- added copper zone on In2.Cu, net +BATT
- added copper zone on B.Cu, net /+12V
- added copper zone on B.Cu, net /+5V
- added copper zone on B.Cu, net GND
- added copper zone on F.Cu, net GND
- added copper zone on In1.Cu, net GND
- added copper zone on F.Cu, net GND1
- added copper zone on In1.Cu, net GND1
- added copper zone on F.Cu, net GND2
- added copper zone on In1.Cu, net GND2
