File: Power management V2/Power_management_V2/Power_management_V2.kicad_pcb (KiCad board)
At the start: 4 copper layers, 76.5 x 66 mm, 58 parts, among them J1 2165711003, U1 SIC43x, U2 SIC43x, U3 TPS3711DDCR

Commit message: Hoan thanh layout va BOM lisst
Parts:
- C24, C6: value 4.7u/16V/1206 -> 4.7u/50V/1206
- C25, C7: value 1u/16V/0603 -> 1u/50V/0603
Other:
- board text added: "0"
- board text added: "0 mm"
- board text added: "0.01 mm"
- board text added: "0.02"
- board text added: "0.061 mm"
- board text added: "0.07 mm"
- board text added: "0.1835 mm"
- board text added: "0.96 mm"
- board text added: "1"
- board text added: "3.3"
- board text added: "4.5"
- board text added: "B.Cu"
- board text added: "B.Mask"
- board text added: "B.Paste"
- board text added: "B.Silkscreen"
- board text added: "Bottom Silk Screen"
- board text added: "Bottom Solder Mask"
- board text added: "Bottom Solder Paste"
- board text added: "Color"
- board text added: "Dielectric 1"
- board text added: "Dielectric 2"
- board text added: "Dielectric 3"
- board text added: "Epsilon R"
- board text added: "F.Cu"
- board text added: "F.Mask"
- board text added: "F.Paste"
- board text added: "F.Silkscreen"
- board text added: "FR4"
- board text added: "In1.Cu"
- board text added: "In2.Cu"
- board text added: "JLC041622-3313(Standard/Finished thickness1.59mm±10%)"
- board text added: "Layer Name"
- board text added: "Loss Tangent"
- board text added: "Material"
- board text added: "Not specified"
- board text added: "Thickness (mm)"
- board text added: "Top Silk Screen"
- board text added: "Top Solder Mask"
- board text added: "Top Solder Paste"
- board text added: "Type"
- board text added: "copper"
- board text added: "core"
- board text added: "prepreg"

Commit message: Cap nhat chiu 3/2
Parts:
- moved C26 41.4 mm to (93.8, 59.6), turned to 90 degrees
- moved C8 31.3 mm to (97.3, 86.3), turned to 90 degrees
- moved C23 4.15 mm to (94.6, 62.7)
- moved R9 4.15 mm to (94.6, 64.2)
- moved C28 4.10 mm to (123.0, 56.5)
- moved C29 4.10 mm to (126.4, 56.5)
- moved C30 4.10 mm to (126.6, 62.9)
- moved C31 4.10 mm to (129.8, 56.4)
- moved NT1 4.10 mm to (99.2, 60.7)
- moved C22 4.10 mm to (99.2, 65.2)
- moved C24 4.10 mm to (102.3, 55.9)
- moved C25 4.10 mm to (98.5, 56.3)
- moved C27 4.10 mm to (123.1, 63.0)
- moved C32 4.10 mm to (133.2, 56.4)
- moved C33 4.10 mm to (136.7, 56.5)
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Routing:
- net Net-(U1-FB): track 7.75 -> 12.5 mm
- net Net-(U1-MODE1): track 7.90 -> 9.33 mm
- net Net-(U1-MODE2): track 6.57 -> 7.41 mm

Commit message: Hoan thanh chinh sua 4/2
Parts:
- removed J1: 2165711003, Library:MOLEX_2165711003
- added J2: 2165711004, Library:MOLEX_2165711004, F.Cu at (144.5, 92.7)
- moved C13 11.2 mm to (136.6, 100.8), turned to -90 degrees
- moved C15 6.57 mm to (133.2, 100.8), turned to -90 degrees
- moved C12 5.81 mm to (115.1, 95.0)
- moved C9 5.81 mm to (115.1, 98.3)
- moved C16 4.47 mm to (122.9, 100.8), turned to -90 degrees
- moved C14 4.32 mm to (126.3, 100.8), turned to -90 degrees
- moved C10 2.69 mm to (129.8, 100.8), turned to -90 degrees
- moved C36 1.63 mm to (119.4, 100.8), turned to -90 degrees
- moved R15 1.54 mm to (144.9, 67.4)
- moved R16 1.46 mm to (147.2, 66.6)
- moved C27 0.67 mm to (123.1, 63.6)
- moved C30 0.67 mm to (126.6, 63.6)
- moved C23 0.46 mm to (94.2, 62.9)
- moved R9 0.46 mm to (94.2, 64.4)
- moved C35 0.08 mm to (135.5, 84.7)
Routing:
- net GND: track 20.8 -> 35.1 mm, vias 136 -> 185
- net /12V/EN_12V: track 118.8 -> 113.5 mm
- net Net-(U1-FB): track 12.5 -> 7.43 mm
- net Net-(U2-MODE2): track 6.27 -> 8.00 mm
- net /+12V: track 34.1 -> 35.7 mm, vias 46 -> 49
- net Net-(U2-MODE1): track 7.61 -> 9.02 mm
- net Net-(U2-PHASE): track 2.32 -> 3.71 mm
- net Net-(U2-BOOT): track 2.04 -> 2.68 mm
- net /+5V: track 35.6 -> 36.1 mm, vias 57 -> 67
- net +BATT: vias 97 -> 96
- net GND2: vias 10 -> 12
- added copper zone on In1.Cu, net +BATT
- added copper zone on In1.Cu, net /+12V
- added copper zone on In1.Cu, net /+5V
- added copper zone on In2.Cu, net /+5V
- added copper zone on In2.Cu, net GND
Other:
- board text added: "12V"
- board text added: "5V"
- board text added: "GND"
- board text removed: "5V 12V GND"
