File: Power management V2/Power_management_V2/Power_management_V2.kicad_pcb (KiCad board)
At the start: 4 copper layers, 76.5 x 66 mm, 58 parts, among them J2 2165711004, U1 SIC43x, U2 SIC43x, U3 TPS3711DDCR

Commit message: Cap Nhat 24/2
Parts:
- added C11: 100n/50V/0603, Capacitor_SMD:C_0603_1608Metric, F.Cu at (124.1, 84.6)
- added C37: 100n/50V/0603, Capacitor_SMD:C_0603_1608Metric, F.Cu at (121.6, 63.7)
- C24, C6: value 4.7u/50V/1206 -> 4.7u/50V/0805; footprint Library:C_1206_3216Metric -> Capacitor_SMD:C_0805_2012Metric
- moved C34 5.52 mm to (148.6, 58.5)
- moved R8 5.52 mm to (145.1, 56.0)
- moved R15 5.52 mm to (145.7, 61.9)
- moved U3 5.52 mm to (145.6, 58.7)
- moved R16 5.52 mm to (148.0, 61.2)
- moved L1 3.12 mm to (115.8, 88.5)
- moved C9 2.66 mm to (116.1, 100.8), turned to -90 degrees
- moved C12 2.39 mm to (113.6, 96.7)
- moved C17 1.16 mm to (133.3, 84.6)
- moved C18 1.16 mm to (130.0, 84.6)
- moved C19 1.16 mm to (126.6, 84.6)
- moved C35 1.16 mm to (136.7, 84.6)
- moved C27 1.07 mm to (124.1, 63.6)
- moved C30 0.88 mm to (127.5, 63.6)
- moved C24 0.52 mm to (101.8, 55.9)
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Routing:
- net /12V/EN_12V: track 113.5 -> 109.9 mm
- net Net-(U2-VDRV): track 6.25 -> 5.14 mm
- net Net-(U1-VDRV): track 5.41 -> 4.86 mm
- net GND: vias 185 -> 189
- net +BATT: vias 96 -> 114
- net GND1: vias 18 -> 20
- net GND2: vias 12 -> 14
- added copper zone on In2.Cu, net /+12V
- removed copper zone on In1.Cu, net /+12V
- removed copper zone on In1.Cu, net /+5V

Commit message: Hoan thanh cap nhat ngay 25/2
Parts:
- J2: value 2165711004 -> 1722861104; footprint Library:MOLEX_2165711004 -> Library:MOLEX_1722861104
- U1, U2: value SIC43x -> SIC437AED
- moved J2 5.22 mm to (139.4, 91.5)
Connections:
- J2 pad 1: /+5V -> /+12V
- J2 pad 4: /+12V -> /+5V
Routing:
- net /+12V: vias 49 -> 47

Commit message: cap nhat 26/2
Changed lines of the file:
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@@
 			(psa4output no)
 			(plot_black_and_white yes)
-			(plotinvisibletext no)
 			(sketchpadsonfab no)
 			(plotpadnumbers no)
@@
 			(pts
 				(xy 119.437786 84.942682) (xy 118.362 86.018468) (xy 118.362 90.8548) (xy 114.642 94.5748) (xy 114.642 99.2098)
-				(xy 116.212 100.7798) (xy 137.732 100.7798) (xy 138.722 99.7898) (xy 138.722 97.8598) (xy 135.3268 94.4646)
-				(xy 135.32325 89.551777) (xy 137.552 87.264113) (xy 137.552 85.091342) (xy 137.387926 84.93058)
+				(xy 116.212 100.7798) (xy 137.732 100.7798) (xy 138.722 99.7898) (xy 138.722 97.8598) (xy 135.880716 95.018516)
+				(xy 135.876356 88.984051) (xy 137.552 87.264113) (xy 137.552 85.091342) (xy 137.387926 84.93058)
 			)
 		)
@@
 		(polygon
 			(pts
-				(xy 120.652 87.8498) (xy 134.84575 87.8498) (xy 135.302 88.30605) (xy 135.302 97.4998) (xy 134.952 97.8498)
+				(xy 120.652 87.8498) (xy 134.84575 87.8498) (xy 135.807 88.81105) (xy 135.807 96.9948) (xy 134.952 97.8498)
 				(xy 120.407 97.8498) (xy 119.952 97.3948) (xy 119.952 88.5498)
 			)
@@
 				(xy 142.152 87.8498) (xy 142.377 88.0748) (xy 142.377 94.6498) (xy 142.877 95.1498) (xy 147.577 95.1498)
 				(xy 147.752 95.3248) (xy 147.752 107.5248) (xy 146.828349 108.448451) (xy 138.900677 108.428973)
-				(xy 135.802 105.322673) (xy 135.802 88.3748) (xy 136.327 87.8498)
+				(xy 136.092 105.613385) (xy 136.092 88.8848) (xy 137.127 87.8498)
 			)
 		)
