File: Power management V2/Power_management_V2/12V.kicad_sch (KiCad schematic)
At the start: 28 parts, among them U1 SIC43x

Commit message: Hoan thanh layout va BOM lisst
Parts:
- C1, C2: JLCPCB Part # (none) -> C508864
- C10, C12, C13, C14, C15, C16, C17, C18, C19, C35, C36, C9: Digikey 445-174338-1-ND -> 1276-3047-1-ND
- C4, C5, C8: JLCPCB Part # (none) -> C1591
- C6: value 4.7u/16V/1206 -> 4.7u/50V/1206; Digikey 490-16469-1-ND -> 490-14384-1-ND; JLCPCB Part # (none) -> C51205; Part GCJ31CL81C475KA01L -> (none)
- C7: value 1u/16V/0603 -> 1u/50V/0603; Digikey 490-GCG188L8EE105KA07DCT-ND -> 1276-1068-1-ND; JLCPCB Part # (none) -> C15849; Part GCG188L8EE105KA07D -> (none)
- L1: Digikey SRP1265A-2R2M -> SRP1265A-2R2MCT-ND
- NT2: Digikey (none) -> NC
- R17: Digikey (none) -> 311-200KHRCT-ND
- U1: Digikey (none) -> SIC437AED-T1-GE3CT-ND

Commit message: Cap Nhat 24/2
Parts:
- added C11: 100n/50V/0603, Capacitor_SMD:C_0603_1608Metric, symbol Device:C
- C10, C12, C13, C14, C15, C16, C17, C18, C19, C35, C36, C9: JLCPCB Part # (none) -> C52306
- C4, C5, C8: JLCPCB Part # C1591 -> C3011652
- C6: value 4.7u/50V/1206 -> 4.7u/50V/0805; footprint Library:C_1206_3216Metric -> Capacitor_SMD:C_0805_2012Metric; Digikey 490-14384-1-ND -> 490-GRM21BZ71H475ME15KCT-ND; JLCPCB Part # C51205 -> C437557
- C7: JLCPCB Part # C15849 -> C5199872
- L1: JLCPCB Part # (none) -> C2831487
- NT2: JLCPCB Part # (none) -> NC
- R17: JLCPCB Part # (none) -> C105574
- R2: JLCPCB Part # (none) -> C144672
- R4, R5: JLCPCB Part # (none) -> C14675
- R6: JLCPCB Part # (none) -> C95204
- R7: JLCPCB Part # (none) -> C861179
- U1: value SIC43x -> SIC437AED; JLCPCB Part # (none) -> C2071432
Connections:
- net GND: now also C11.1
- net VOUT_12V: now also C11.2
