File: Power management V2/Power_management_V2/5V.kicad_sch (KiCad schematic)
At the start: 23 parts, among them U2 SIC43x

Commit message: Hoan thanh layout va BOM lisst
Parts:
- C20, C21: JLCPCB Part # (none) -> C508864
- C22, C23, C26: JLCPCB Part # (none) -> C1591
- C24: value 4.7u/16V/1206 -> 4.7u/50V/1206; Digikey 490-16469-1-ND -> 490-14384-1-ND; JLCPCB Part # (none) -> C51205; Part GCJ31CL81C475KA01L -> (none)
- C25: value 1u/16V/0603 -> 1u/50V/0603; Digikey 490-GCG188L8EE105KA07DCT-ND -> 1276-1068-1-ND; JLCPCB Part # (none) -> C15849; Part GCG188L8EE105KA07D -> (none)
- C27, C28, C29, C30, C31, C32, C33: Digikey 445-174338-1-ND -> 1276-3047-1-ND
- L2: Digikey SRP1265A-2R2M -> SRP1265A-2R2MCT-ND
- NT1: Digikey (none) -> NC
- R10: Digikey (none) -> 311-200KHRCT-ND
- R14: Digikey (none) -> P73.2KDBCT-ND

Commit message: Cap Nhat 24/2
Parts:
- added C37: 100n/50V/0603, Capacitor_SMD:C_0603_1608Metric, symbol Device:C
- C22, C23, C26: JLCPCB Part # C1591 -> C3011652
- C24: value 4.7u/50V/1206 -> 4.7u/50V/0805; footprint Library:C_1206_3216Metric -> Capacitor_SMD:C_0805_2012Metric; Coefficient X8L -> (none); Digikey 490-14384-1-ND -> 490-GRM21BZ71H475ME15KCT-ND; JLCPCB Part # C51205 -> C437557; Tolerance 10 -> (none); Voltage 16 -> (none)
- C25: JLCPCB Part # C15849 -> C5199872
- C27, C28, C29, C30, C31, C32, C33: JLCPCB Part # (none) -> C52306
- L2: JLCPCB Part # (none) -> C2831487
- NT1: JLCPCB Part # (none) -> NC
- R10: JLCPCB Part # (none) -> C105574
- R11, R12: JLCPCB Part # (none) -> C14675
- R13: JLCPCB Part # (none) -> C95204
- R14: JLCPCB Part # (none) -> C862276
- R9: JLCPCB Part # (none) -> C144672
- U2: value SIC43x -> SIC437AED; JLCPCB Part # (none) -> C2071432
Connections:
- net GND: now also C37.1
- net VOUT: now also C37.2
