File: Connector Extension Board V1.0/Connector_Extension_Board_V1.0/Connector_Extension_Board_V1.0.kicad_pcb (KiCad board)
At the start: 4 copper layers, 67.7 x 69 mm, 63 parts, among them J1 2157601003, U10 TPS259571DSGR, U11 TPS259571DSGR, U12 TPS259571DSGR, U3 TPS259571DSGR, U4 TPS259571DSGR, U5 TPS259571DSGR, U8 TPS259571DSGR, U9 TPS1HC30BQPWPRQ1

Commit message: Hoan thanh layout va BOM lisst
Parts:
- added H1: MountingHole_Pad, Library:MountingHole_3.1-5.8, F.Cu at (113.0, 52.5)
- added H2: MountingHole_Pad, Library:MountingHole_3.1-5.8, F.Cu at (162.5, 114.5)
- added H3: MountingHole_Pad, Library:MountingHole_3.1-5.8, F.Cu at (103.5, 114.5)
- C26, C8: value 100nF/50V/0603 -> 100n/50V/0603
- GPS1, Phone1: value Conn_01x02 -> 5-104361-1
- moved C26 0.20 mm to (155.5, 98.1)
Routing:
- net /V_EN: track 0.00 -> 103.2 mm, vias 0 -> 8
- net +5V: track 0.00 -> 47.2 mm, vias 0 -> 70
- net Net-(U5-DVDT): track 0.00 -> 4.22 mm
- net Net-(U9-SNS): track 0.00 -> 3.60 mm
- net Net-(U10-DVDT): track 0.00 -> 3.44 mm
- net Net-(U8-DVDT): track 0.00 -> 3.34 mm
- net Net-(U4-DVDT): track 0.00 -> 3.34 mm
- net Net-(U11-DVDT): track 0.00 -> 3.34 mm
- net Net-(U12-DVDT): track 0.00 -> 3.01 mm
- net Net-(U8-ILM): track 0.00 -> 2.93 mm
- net Net-(U5-ILM): track 0.00 -> 2.93 mm
- net Net-(U4-ILM): track 0.00 -> 2.93 mm
- net Net-(U11-ILM): track 0.00 -> 2.93 mm
- net Net-(U9-LATCH): track 0.00 -> 2.77 mm
- net Net-(U9-EN): track 0.00 -> 2.72 mm
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- added copper zone on B.Cu, net +12V
- added copper zone on F.Cu, net +12V
- added copper zone on In1.Cu, net +12V
- added copper zone on In2.Cu, net +12V
- added copper zone on B.Cu, net +5V
- added copper zone on F.Cu, net +5V
- added copper zone on In1.Cu, net +5V
- added copper zone on In2.Cu, net +5V
- added copper zone on F.Cu, net /+12V-0.2A
- added copper zone on F.Cu, net /+12V-1A
- added copper zone on F.Cu, net /+12V-2.5A
- added copper zone on F.Cu, net /+12V-3A
- added copper zone on B.Cu, net /+12V-7A
- added copper zone on F.Cu, net /+12V-7A
- added copper zone on F.Cu, net /+5V-2A
- added copper zone on F.Cu, net /+5V-3A_1
- added copper zone on F.Cu, net /+5V-3A_2
- added copper zone on B.Cu, net GND
- added copper zone on F.Cu, net GND
Other:
- board text added: "-"
- board text added: "0"
- board text added: "0 mm"
- board text added: "0.01 mm"
- board text added: "0.02"
- board text added: "0.061 mm"
- board text added: "0.07 mm"
- board text added: "0.1835 mm"
- board text added: "0.96 mm"
- board text added: "1"
- board text added: "3.3"
- board text added: "4.5"
- board text added: "B.Cu"
- board text added: "B.Mask"
- board text added: "B.Paste"
- board text added: "B.Silkscreen"
- board text added: "Bottom Silk Screen"
- board text added: "Bottom Solder Mask"
- board text added: "Bottom Solder Paste"
- board text added: "Color"
- board text added: "Dielectric 1"
- board text added: "Dielectric 2"
- board text added: "Dielectric 3"
- board text added: "Epsilon R"
- board text added: "F.Cu"
- board text added: "F.Mask"
- board text added: "F.Paste"
- board text added: "F.Silkscreen"
- board text added: "FR4"
- board text added: "In1.Cu"
- board text added: "In2.Cu"
- board text added: "JLC041622-3313(Standard/Finished thickness1.59mm±10%)"
- board text added: "Layer Name"
- board text added: "Loss Tangent"
- board text added: "Material"
- board text added: "Not specified"
- board text added: "Thickness (mm)"
- board text added: "Top Silk Screen"
- board text added: "Top Solder Mask"
- board text added: "Top Solder Paste"
- board text added: "Type"
- board text added: "copper"
- board text added: "core"
- board text added: "prepreg"

Commit message: Hoan thanh chinh sua 4/2
Parts:
- removed R24: 10k/0603/1%, Resistor_SMD:R_0603_1608Metric
- J1: footprint Library:MOLEX_2157601003 -> Library:MOLEX_2157601004
- moved R44 26.5 mm to (143.4, 78.8), turned to 180 degrees
- moved R14 25.9 mm to (146.5, 78.8)
- moved C5 1.46 mm to (138.5, 88.6)
- moved C9 1.46 mm to (139.3, 90.7)
- moved C26 1.40 mm to (156.9, 98.1)
- moved C21 1.39 mm to (116.5, 97.1)
- moved C27 1.39 mm to (126.8, 97.1)
- moved C16 1.38 mm to (138.6, 97.0)
- moved C19 1.38 mm to (105.2, 97.0)
- moved C28 1.36 mm to (155.5, 80.1)
- moved C15 1.30 mm to (149.5, 73.2)
- moved C22 1.27 mm to (105.3, 78.2)
- moved C13 1.25 mm to (106.2, 91.3)
- moved C10 1.20 mm to (127.8, 90.7)
- moved C7 1.20 mm to (127.0, 88.7)
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Connections:
- J1 pad 2: +12V -> GND
- U9 pad 4: Net-(U9-~{FAULT}) -> unconnected-(U9-~{FAULT}-Pad4)
Routing:
- net +5V: track 47.2 -> 9.94 mm, vias 70 -> 69
- net /V_EN: track 103.2 -> 78.3 mm, vias 8 -> 6
- net +12V: track 2.02 -> 9.30 mm, vias 116 -> 97
- net Net-(U9-~{FAULT}): track 2.34 -> 0.00 mm
- net GND: vias 178 -> 212
- added copper zone on In1.Cu, net GND
- added copper zone on In2.Cu, net GND
- removed copper zone on In1.Cu, net +12V
- removed copper zone on In2.Cu, net +12V
- removed copper zone on In1.Cu, net +5V
- removed copper zone on In2.Cu, net +5V
Other:
- board text added: "5V GND GND 12V"
- board text removed: "5V 12V GND"

Commit message: Cap Nhat 24/2
Changed lines of the file:
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@@
 		(at 130.7045 93.3573 -90)
 		(property "Reference" "U5"
-			(at 0.547 -1.9564 270)
+			(at 0.0675 -2.2725 0)
 			(layer "F.SilkS")
 			(effects
@@
 		(at 159.052 77.0673 -90)
 		(property "Reference" "U10"
-			(at -0.0175 -1.9 270)
+			(at 0.0575 -2.525 0)
 			(layer "F.SilkS")
 			(effects
@@
 		(tags "resistor")
 		(property "Reference" "R26"
-			(at -2.975 0.13 90)
+			(at -2.975 -0.005 90)
 			(layer "F.SilkS")
 			(effects
@@
 		(at 145.6745 69.3698)
 		(property "Reference" "U3"
-			(at 0.547 -1.9564 0)
+			(at 0.0275 -2.02 0)
 			(layer "F.SilkS")
 			(effects
@@
 		(pad "" np_thru_hole circle
 			(at -1.47 -8.64 180)
-			(size 2.36 2.36)
-			(drill 2.36)
+			(size 2.4 2.36)
+			(drill 2.4)
 			(layers "*.Cu" "*.Mask")
 		)
 		(pad "" np_thru_hole circle
 			(at 4.01 -8.64 180)
-			(size 2.36 2.36)
-			(drill 2.36)
+			(size 2.4 2.36)
+			(drill 2.4)
 			(layers "*.Cu" "*.Mask")
 		)
 		(pad "1" thru_hole rect
 			(at 0 0 180)
-			(size 1.78 1.78)
+			(size 1.8 1.8)
 			(drill 1)
 			(layers "*.Cu" "*.Mask")
@@
 		(pad "2" thru_hole circle
 			(at 2.54 0 180)
-			(size 1.75 1.75)
+			(size 1.75 1.8)
 			(drill 1)
 			(layers "*.Cu" "*.Mask")
@@
 		(tags "capacitor")
 		(property "Reference" "C21"
-			(at 0.8 1.78 0)
+			(at 0.845 1.835 0)
 			(layer "F.SilkS")
 			(effects
@@
 		(tags "capacitor")
 		(property "Reference" "C19"
-			(at -0.06 -1.91 0)
+			(at 0.045 1.825 0)
 			(layer "F.SilkS")
 			(effects
@@
 		(tags "capacitor")
 		(property "Reference" "C4"
-			(at 0.07 1.71 90)
+			(at 3.475 0 90)
 			(layer "F.SilkS")
 			(effects
@@
 		(at 120.242 93.3673 -90)
 		(property "Reference" "U11"
-			(at 0.547 -1.9564 270)
+			(at -0.0175 -2.61 0)
 			(layer "F.SilkS")
 			(effects
@@
 		(tags "capacitor")
 		(property "Reference" "C6"
-			(at 3.34 0 0)
+			(at -0.01 1.86 0)
 			(layer "F.SilkS")
 			(effects
@@
 		(at 153.382 93.1198 -90)
 		(property "Reference" "U9"
-			(at 0.34 -3.56 90)
+			(at 0.255 -4.245 180)
 			(layer "F.SilkS")
 			(effects
@@
 			(at 0 0)
 			(size 2 2)
-			(drill 1.02)
+			(drill 1.05)
 			(layers "*.Cu")
 			(remove_unused_layers no)
@@
 			(at 3.5 0)
 			(size 2 2)
-			(drill 1.02)
+			(drill 1.05)
 			(layers "*.Cu")
 			(remove_unused_layers no)
@@
 		(pad "4" thru_hole circle
 			(at -2.5 7.91)
-			(size 2.2606 2.2606)
-			(drill 1.7526)
+			(size 2.3 2.2606)
+			(drill 1.8)
 			(layers "*.Cu" "*.Mask")
 			(remove_unused_layers no)
@@
 		(pad "5" thru_hole circle
 			(at 6 7.91)
-			(size 2.2606 2.2606)
-			(drill 1.7526)
+			(size 2.3 2.2606)
+			(drill 1.8)
 			(layers "*.Cu" "*.Mask")
 			(remove_unused_layers no)
@@
 		(tags "capacitor")
 		(property "Reference" "C16"
-			(at 1.45 1.71 180)
+			(at 1.495 1.805 180)
 			(layer "F.SilkS")
 			(effects
@@
 			(at 0 0 180)
 			(size 2 2)
-			(drill 1.02)
+			(drill 1.05)
 			(layers "*.Cu")
 			(remove_unused_layers no)
@@
 			(at 3.5 0 180)
 			(size 2 2)
-			(drill 1.02)
+			(drill 1.05)
 			(layers "*.Cu")
 			(remove_unused_layers no)
@@
 		(pad "4" thru_hole circle
 			(at -2.5 7.91 180)
-			(size 2.2606 2.2606)
-			(drill 1.7526)
+			(size 2.3 2.2606)
+			(drill 1.8)
 			(layers "*.Cu" "*.Mask")
 			(remove_unused_layers no)
@@
 		(pad "5" thru_hole circle
 			(at 6 7.91 180)
-			(size 2.2606 2.2606)
-			(drill 1.7526)
+			(size 2.3 2.2606)
+			(drill 1.8)
 			(layers "*.Cu" "*.Mask")
 			(remove_unused_layers no)
@@
 		(tags "resistor")
 		(property "Reference" "R27"
-			(at -2.855 0.34 90)
+			(at -3.035 -0.015 90)
 			(layer "F.SilkS")
 			(effects
@@
 		(tags "resistor")
 		(property "Reference" "R28"
-			(at -2.995 0.1 90)
+			(at -3.02 -0.015 90)
 			(layer "F.SilkS")
 			(effects
@@
 		(at 108.892 75.5273 -90)
 		(property "Reference" "U12"
-			(at -0.3775 -1.95 270)
+			(at 0.0475 -2.585 0)
 			(layer "F.SilkS")
 			(effects
@@
 			(at 0 0)
 			(size 2 2)
-			(drill 1.02)
+			(drill 1.05)
 			(layers "*.Cu")
 			(remove_unused_layers no)
@@
 			(at 3.5 0)
 			(size 2 2)
-			(drill 1.02)
+			(drill 1.05)
 			(layers "*.Cu")
 			(remove_unused_layers no)
@@
 		(pad "4" thru_hole circle
 			(at -2.5 7.91)
-			(size 2.2606 2.2606)
-			(drill 1.7526)
+			(size 2.3 2.2606)
+			(drill 1.8)
 			(layers "*.Cu" "*.Mask")
 			(remove_unused_layers no)
@@
 		(pad "5" thru_hole circle
 			(at 6 7.91)
-			(size 2.2606 2.2606)
-			(drill 1.7526)
+			(size 2.3 2.2606)
+			(drill 1.8)
 			(layers "*.Cu" "*.Mask")
 			(remove_unused_layers no)
@@
 		(tags "capacitor")
 		(property "Reference" "C27"
-			(at 1.72 1.8 0)
+			(at 1.765 1.855 0)
 			(layer "F.SilkS")
 			(effects
@@
 			(at 0 0)
 			(size 2 2)
-			(drill 1.02)
+			(drill 1.05)
 			(layers "*.Cu")
 			(remove_unused_layers no)
@@
 			(at 3.5 0)
 			(size 2 2)
-			(drill 1.02)
+			(drill 1.05)
 			(layers "*.Cu")
 			(remove_unused_layers no)
@@
 		(pad "4" thru_hole circle
 			(at -2.5 7.91)
-			(size 2.2606 2.2606)
-			(drill 1.7526)
+			(size 2.3 2.2606)
+			(drill 1.8)
 			(layers "*.Cu" "*.Mask")
 			(remove_unused_layers no)
@@
 		(pad "5" thru_hole circle
 			(at 6 7.91)
-			(size 2.2606 2.2606)
-			(drill 1.7526)
+			(size 2.3 2.2606)
+			(drill 1.8)
 			(layers "*.Cu" "*.Mask")
 			(remove_unused_layers no)
@@
 		(pad "" np_thru_hole circle
 			(at -1.47 -8.64 180)
-			(size 2.36 2.36)
-			(drill 2.36)
+			(size 2.4 2.36)
+			(drill 2.4)
 			(layers "*.Cu" "*.Mask")
 		)
 		(pad "" np_thru_hole circle
 			(at 4.01 -8.64 180)
-			(size 2.36 2.36)
-			(drill 2.36)
-			(layers "*.Cu" "*.Mask")
+			(size 2.4 2.4)
+			(drill 2.4)
+			(layers "F&B.Cu" "*.Mask")
 		)
 		(pad "1" thru_hole rect
 			(at 0 0 180)
-			(size 1.78 1.78)
+			(size 1.8 1.8)
 			(drill 1)
 			(layers "*.Cu" "*.Mask")
@@
 		(pad "2" thru_hole circle
 			(at 2.54 0 180)
-			(size 1.75 1.75)
+			(size 1.75 1.8)
 			(drill 1)
 			(layers "*.Cu" "*.Mask")
@@
 		(at 109.002 93.3673 -90)
 		(property "Reference" "U8"
-			(at 0.547 -1.9564 270)
+			(at 0.1325 -2.1 0)
 			(layer "F.SilkS")
 			(effects
@@
 		(tags "capacitor")
 		(property "Reference" "C13"
-			(at 2.35 -4.22 0)
+			(at 3.022239 0.007924 0)
 			(layer "F.SilkS")
 			(effects
@@
 		(tags "resistor")
 		(property "Reference" "R25"
-			(at 3.085 -0.07 90)
+			(at 2.99 0.025 90)
 			(layer "F.SilkS")
 			(effects
@@
 		(tags "capacitor")
 		(property "Reference" "C11"
-			(at 1.58 -3.71 0)
+			(at 2.925 0 0)
 			(layer "F.SilkS")
 			(effects
@@
 			(effects
 				(font
-					(size 1 1)
-					(thickness 0.15)
+					(size 0.8 0.8)
+					(thickness 0.2)
 				)
 			)
@@
 		(pad "1" thru_hole rect
 			(at 0 0 180)
-			(size 1.52 1.52)
-			(drill 1.02)
+			(size 1.5 1.52)
+			(drill 1.05)
 			(layers "*.Cu")
 			(remove_unused_layers no)
@@
 		(pad "2" thru_hole circle
 			(at -3 0 180)
-			(size 1.52 1.52)
-			(drill 1.02)
+			(size 1.5 1.52)
+			(drill 1.05)
 			(layers "*.Cu")
 			(remove_unused_layers no)
@@
 		(pad "3" thru_hole circle
 			(at -6 0 180)
-			(size 1.52 1.52)
-			(drill 1.02)
+			(size 1.5 1.52)
+			(drill 1.05)
 			(layers "*.Cu")
 			(remove_unused_layers no)
@@
 		(pad "4" thru_hole circle
 			(at -9 0 180)
-			(size 1.52 1.52)
-			(drill 1.02)
+			(size 1.5 1.52)
+			(drill 1.05)
 			(layers "*.Cu")
 			(remove_unused_layers no)
@@
 		(at 142.302 93.3573 -90)
 		(property "Reference" "U4"
-			(at 0 1.85 90)
+			(at 0 -2.95 180)
 			(layer "F.SilkS")
 			(effects
@@
 	)
 	(gr_text "Spare"
-		(at 127.162 100.2598 0)
+		(at 127.162 100.3198 0)
 		(layer "F.SilkS")
 		(effects
@@
 	)
 	(gr_text "Phone\n"
-		(at 116.912 101.5398 0)
+		(at 116.772 101.5898 0)
 		(layer "F.SilkS")
 		(effects
@@
 	)
 	(gr_text "Winch"
-		(at 150.562 100.5298 0)
+		(at 150.562 100.3198 0)
 		(layer "F.SilkS")
 		(effects
@@
 	)
 	(gr_text "LoRa "
-		(at 164.452 87.0998 90)
+		(at 164.477 87.2498 90)
 		(layer "F.SilkS")
 		(effects

Commit message: Hoan thanh cap nhat ngay 25/2
Parts:
- J1: value 2157601003 -> 1723103104; footprint Library:MOLEX_2157601004 -> Library:MOLEX_1723103104
- moved J1 4.66 mm to (128.8, 58.3)
- moved C28 0.70 mm to (155.5, 79.4)
Connections:
- J1 pad 1: +5V -> +12V
- J1 pad 4: +12V -> +5V

Commit message: cap nhat 26/2
Changed lines of the file:
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@@
 			(disableapertmacros no)
 			(usegerberextensions yes)
-			(usegerberattributes yes)
+			(usegerberattributes no)
 			(usegerberadvancedattributes no)
 			(creategerberjobfile no)
@@
 			(psa4output no)
 			(plot_black_and_white yes)
-			(plotinvisibletext no)
 			(sketchpadsonfab no)
 			(plotpadnumbers no)
@@
 			(pinfunction "Pin_2")
 			(pintype "passive")
+			(zone_connect 1)
+			(thermal_bridge_width 0.8)
+			(thermal_gap 0.3)
 		)
 		(pad "3" thru_hole circle
@@
 			(pinfunction "Pin_3")
 			(pintype "passive")
+			(zone_connect 1)
+			(thermal_bridge_width 0.8)
+			(thermal_gap 0.3)
 		)
 		(pad "4" thru_hole circle
@@
 		(hatch edge 0.5)
 		(connect_pads
-			(clearance 0.4)
+			(clearance 0.5)
 		)
 		(min_thickness 0.2)
@@
 		(layer "F.Cu")
 		(hatch edge 0.5)
+		(priority 1)
 		(connect_pads
 			(clearance 0.3)
@@
 		(polygon
 			(pts
-				(xy 132.352 75.6998) (xy 127.3045 80.7473) (xy 127.3045 86.5148) (xy 127.7895 86.9998) (xy 131.4345 86.9998)
+				(xy 132.072 75.9798) (xy 127.3045 80.7473) (xy 127.3045 86.5148) (xy 127.7895 86.9998) (xy 131.4345 86.9998)
 				(xy 131.4795 87.0448) (xy 143.052 87.0448) (xy 143.052 77.4273) (xy 142.6245 76.9998) (xy 140.852 76.9998)
 				(xy 139.752 75.8998) (xy 139.752 72.2098) (xy 140.552 71.4098) (xy 140.552 68.0498) (xy 139.052 66.5498)
-				(xy 139.052 60.9498) (xy 138.302 60.1998) (xy 133.102 60.1998) (xy 132.352 60.9498)
+				(xy 139.052 60.9498) (xy 138.302 60.1998) (xy 133.102 60.1998) (xy 132.072 61.2298)
 			)
 		)
@@
 				(xy 114.102 72.3498) (xy 114.102 80.283133) (xy 113.852 80.6998) (xy 109.702 80.6998) (xy 105.602 84.7998)
 				(xy 105.602 86.5498) (xy 106.452 87.3998) (xy 122.034402 87.308139) (xy 123.377 86.099801) (xy 123.377 75.763631)
-				(xy 125.234783 73.233883) (xy 125.234783 61.432583) (xy 123.978596 60.176396)
+				(xy 125.474783 72.907075) (xy 125.474783 61.672583) (xy 123.978596 60.176396)
 			)
 		)
@@
 		(polygon
 			(pts
-				(xy 132.152 60.6498) (xy 132.152 74.2998) (xy 127.252 79.1998) (xy 127.252 86.5998) (xy 129.452 88.7998)
+				(xy 132.242 60.5598) (xy 132.242 74.2098) (xy 127.252 79.1998) (xy 127.252 86.5998) (xy 129.452 88.7998)
 				(xy 144.452 88.7998) (xy 154.652 88.7998) (xy 156.852 90.9998) (xy 156.852 94.4998) (xy 153.752 97.5998)
 				(xy 153.752 101.2998) (xy 153.952 101.4998) (xy 165.150171 101.4998) (xy 165.848043 100.801928)
